Commit message: feat: tmr v02 added to franka description

File: robots/tmr/argo_drive.xacro (robot description, xacro)
@@ -2,12 +2,13 @@
 <robot xmlns:xacro="http://www.ros.org/wiki/xacro" >
   <xacro:include filename="$(find franka_description)/robots/tmr/inertia.xacro" />
-  <xacro:macro name="caster_wheel" params="name parent length:='0.015' radius:='0.03' caster_joint_z:='-0.05' caster_steering_offset:='-0.035' *origin">
-    <xacro:property name="base_width" value="0.04" />
-    <xacro:property name="base_depth" value="0.03" />
-    <xacro:property name="base_height" value="0.003" />
+  <xacro:macro name="argo_drive" params="name parent length:='0.04' radius:='0.05' offset_wheel_sign:='1' *origin">
+    <xacro:property name="base_width" value="0.17" />
+    <xacro:property name="base_depth" value="0.25" />
+    <xacro:property name="base_height" value="0.077" />
+    <xacro:property name="offset_wheel" value="0.085" />
     <xacro:property name="mass" value="0.5" />
     <link name="${name}_fixed_link" >
       <xacro:macro name="caster_base_geometry" params="xyz:='0 0 0'">
-        <origin xyz="0 0 ${-base_height/2}" />
+        <origin xyz="0 ${offset_wheel_sign*(base_depth/2 - offset_wheel)} ${base_height/2 - 0.004}" />
         <geometry>
           <box size="${base_width} ${base_depth} ${base_height}" />
@@ -39,23 +40,23 @@
     </joint>
     <link name="${name}_link" >
-      <xacro:macro name="caster_wheel_geometry">
+      <xacro:macro name="argo_drive_geometry">
         <origin rpy="${pi/2} 0 0" />
         <geometry>
            <cylinder length="${length}" radius="${radius}" />
         </geometry>
-        <material name="orange">
-          <color rgba="1.0 0.5 0.0 1.0"/>
+        <material name="yellowish_brown">
+          <color rgba="0.8 0.6 0.2 1.0"/>
         </material>
       </xacro:macro>
       <visual>
-        <xacro:caster_wheel_geometry/>
+        <xacro:argo_drive_geometry/>
       </visual>
       <collision>
-        <xacro:caster_wheel_geometry/>
+        <xacro:argo_drive_geometry/>
       </collision>
       <xacro:inertia-cylinder mass="${mass}" radius="${radius}" h="${length}" />
     </link>
     <joint name="${name}_joint" type="continuous">
-      <origin xyz ="${caster_steering_offset} 0 ${caster_joint_z}" rpy="0 0 0" />
+      <origin xyz ="0 0 0" rpy="0 0 0" />
       <parent link="${name}_steering_link" />
       <child  link="${name}_link" />

File: robots/tmr/rocker_arm.xacro (robot description, xacro)
@@ -2,5 +2,5 @@
 <robot xmlns:xacro="http://www.ros.org/wiki/xacro" >
   <xacro:include filename="$(find franka_description)/robots/tmr/inertia.xacro" />
-  <xacro:macro name="bogie" params="name mass parent *origin">
+  <xacro:macro name="rocker_arm" params="name mass parent *origin">
     <xacro:property name="depth" value="0.32"/>
     <xacro:property name="width" value="0.02"/>
@@ -8,5 +8,5 @@
     <link name="${name}_link" >
       <visual>
-        <origin rpy="${pi/2} 0 0" />
+        <origin rpy="${pi/2} 0 ${pi/2}" />
         <geometry>
           <cylinder radius="${height}" length="${height*1.5}" />
@@ -24,5 +24,5 @@
       <parent link="${parent}" />
       <child  link="${name}_link" />
-      <axis   xyz="0 1 0" />
+      <axis   xyz="1 0 0" />
       <limit  effort="500" velocity="20" upper="0.18" lower="-0.16"/>
       <dynamics damping="0.003" friction="0.0"/>
