Commit message: chore: tmr v02 files renamed

File: robots/common/franka_arm.ros2_control.xacro (robot description, xacro)
@@ -61,5 +61,4 @@
         <xacro:configure_joint joint_name="${arm_prefix}${arm_id}_finger_joint1" initial_position="0.0" />
       </xacro:if>
-      <!-- General purpose IO interfaces -->
       <xacro:macro name="general_purpose_io" params="prefix command_interface index">
         <gpio name="${prefix}">
@@ -69,15 +68,14 @@
       </xacro:macro>
       <!-- Cartesian velocity interfaces -->
-      <xacro:property name="gpios_suffix" value="${'' if arm_prefix == '' else arm_prefix_modified + arm_id + '_'}" />
-      <xacro:general_purpose_io prefix="${gpios_suffix}vx" command_interface="cartesian_velocity" index="0"/>
-      <xacro:general_purpose_io prefix="${gpios_suffix}vy" command_interface="cartesian_velocity" index="1"/>
-      <xacro:general_purpose_io prefix="${gpios_suffix}vz" command_interface="cartesian_velocity" index="2"/>
-      <xacro:general_purpose_io prefix="${gpios_suffix}wx" command_interface="cartesian_velocity" index="3"/>
-      <xacro:general_purpose_io prefix="${gpios_suffix}wy" command_interface="cartesian_velocity" index="4"/>
-      <xacro:general_purpose_io prefix="${gpios_suffix}wz" command_interface="cartesian_velocity" index="5"/>
+      <xacro:general_purpose_io prefix="vx" command_interface="cartesian_velocity" index="0"/>
+      <xacro:general_purpose_io prefix="vy" command_interface="cartesian_velocity" index="1"/>
+      <xacro:general_purpose_io prefix="vz" command_interface="cartesian_velocity" index="2"/>
+      <xacro:general_purpose_io prefix="wx" command_interface="cartesian_velocity" index="3"/>
+      <xacro:general_purpose_io prefix="wy" command_interface="cartesian_velocity" index="4"/>
+      <xacro:general_purpose_io prefix="wz" command_interface="cartesian_velocity" index="5"/>
       <!-- Cartesian pose interfaces, in total 16 interfaces -->
       <xacro:macro name="loop" params="i">
         <xacro:unless value="${i == 16}">
-          <xacro:general_purpose_io prefix="${gpios_suffix}${i}" command_interface="cartesian_pose_command" index="${i}"/>
+          <xacro:general_purpose_io prefix="${i}" command_interface="cartesian_pose_command" index="${i}"/>
           <xacro:loop i="${i+1}"/>
         </xacro:unless>
@@ -85,6 +83,6 @@
       <xacro:loop i="0"/>
       <!-- Elbow command interfaces -->
-      <xacro:general_purpose_io prefix="${gpios_suffix}joint_3_position" command_interface="elbow_command" index="0"/>
-      <xacro:general_purpose_io prefix="${gpios_suffix}joint_4_sign" command_interface="elbow_command" index="1"/>
+      <xacro:general_purpose_io prefix="joint_3_position" command_interface="elbow_command" index="0"/>
+      <xacro:general_purpose_io prefix="joint_4_sign" command_interface="elbow_command" index="1"/>
     </ros2_control>
     <xacro:if value="${gazebo}">

File: robots/tmr_v02/argo_drive.xacro (robot description, xacro)
@@ -1,5 +1,5 @@
 <?xml version="1.0"?>
 <robot xmlns:xacro="http://www.ros.org/wiki/xacro" >
-  <xacro:include filename="$(find franka_description)/robots/tmr/inertia.xacro" />
+  <xacro:include filename="$(find franka_description)/robots/tmr_v02/inertia.xacro" />
   <xacro:macro name="argo_drive" params="name parent length:='0.04' radius:='0.05' offset_wheel_sign:='1' *origin">
     <xacro:property name="base_width" value="0.17" />

File: robots/tmr_v02/caster_wheel.xacro (robot description, xacro)
@@ -1,5 +1,5 @@
 <?xml version="1.0"?>
 <robot xmlns:xacro="http://www.ros.org/wiki/xacro" >
-  <xacro:include filename="$(find franka_description)/robots/tmr/inertia.xacro" />
+  <xacro:include filename="$(find franka_description)/robots/tmr_v02/inertia.xacro" />
   <xacro:macro name="caster_wheel" params="name parent length:='0.015' radius:='0.03' caster_joint_z:='-0.05' caster_steering_offset:='-0.035' *origin">
     <xacro:property name="base_width" value="0.04" />

File: robots/tmr_v02/lidar.xacro (robot description, xacro)
@@ -2,5 +2,5 @@
 <robot xmlns:xacro="http://www.ros.org/wiki/xacro" >
   <xacro:macro name="lidar" params="name parent min_angle:='${radians(-45)}' max_angle:='${radians(225)}' *origin ">
-    <xacro:include filename="$(find franka_description)/robots/tmr/nanoscan3/nanoscan3/nanoscan3_macro.xacro"/>
+    <xacro:include filename="$(find franka_description)/robots/tmr_v02/nanoscan3/nanoscan3/nanoscan3_macro.xacro"/>
     <xacro:nanoscan3
       name="${name}"

File: robots/tmr_v02/nanoscan3/nanoscan3.urdf.xacro (robot description, xacro)
@@ -8,5 +8,5 @@
   <!-- Load robot's macro with parameters -->
   <!-- set prefix if multiple robots are used -->
-  <xacro:include filename="$(find sick_safetyscanners2)/description/robots/tmr/nanoscan3/nanoscan3_macro.xacro"/>
+  <xacro:include filename="$(find sick_safetyscanners2)/description/robots/tmr_v02/nanoscan3/nanoscan3_macro.xacro"/>
   <xacro:property name="mounting_kit" value="$(arg mounting_kit)"/>
   <xacro:nanoscan3

File: robots/tmr_v02/nanoscan3/nanoscan3/nanoscan3_macro.xacro (robot description, xacro)
@@ -1,6 +1,6 @@
 <?xml version="1.0" encoding="UTF-8"?>
 <robot xmlns:xacro="http://wiki.ros.org/xacro">
-  <xacro:include filename="$(find franka_description)/robots/tmr/nanoscan3/common.xacro" />
-  <xacro:include filename="$(find franka_description)/robots/tmr/nanoscan3/nanoscan3/gazebo_macro.xacro" />
+  <xacro:include filename="$(find franka_description)/robots/tmr_v02/nanoscan3/common.xacro" />
+  <xacro:include filename="$(find franka_description)/robots/tmr_v02/nanoscan3/nanoscan3/gazebo_macro.xacro" />
   <!-- joint offsets when mounted on frame -->
   <xacro:property name="base_x" value="0.0803"/>

File: robots/tmr_v02/rocker_arm.xacro (robot description, xacro)
@@ -1,5 +1,5 @@
 <?xml version="1.0"?>
 <robot xmlns:xacro="http://www.ros.org/wiki/xacro" >
-  <xacro:include filename="$(find franka_description)/robots/tmr/inertia.xacro" />
+  <xacro:include filename="$(find franka_description)/robots/tmr_v02/inertia.xacro" />
   <xacro:macro name="rocker_arm" params="name mass parent *origin">
     <xacro:property name="depth" value="0.32"/>

File: robots/tmr_v02/tmr_v02.ros2_control.xacro (robot description, xacro)
@@ -1,5 +1,5 @@
 <?xml version="1.0"?>
 <robot xmlns:xacro="http://www.ros.org/wiki/xacro">
-  <xacro:macro name="tmr_ros2_control"
+  <xacro:macro name="tmr_v02_ros2_control"
     params="mobile_robot_id
             robot_ip
@@ -10,5 +10,5 @@
         <param name="version">0.1.0</param>
         <param name="mobile_robot_id">${mobile_robot_id}</param>
-        <param name="arm_id">tmr</param>
+        <param name="arm_id">tmr_v02</param>
         <xacro:if value="${use_fake_hardware}">
           <plugin>fake_components/GenericSystem</plugin>

File: robots/tmr_v02/tmr_v02.xacro (robot description, xacro)
@@ -1,5 +1,5 @@
 <?xml version="1.0"?>
 <robot xmlns:xacro="http://www.ros.org/wiki/xacro">
-  <xacro:macro name="tmr"
+  <xacro:macro name="tmr_v02"
     params="mobile_robot_id
                   robot_ip:=''
@@ -7,9 +7,9 @@
                   use_fake_hardware:=false
                   fake_sensor_commands:=false">
-    <xacro:include filename="$(find franka_description)/robots/tmr/argo_drive.xacro" />
-    <xacro:include filename="$(find franka_description)/robots/tmr/caster_wheel.xacro" />
-    <xacro:include filename="$(find franka_description)/robots/tmr/rocker_arm.xacro" />
-    <xacro:include filename="$(find franka_description)/robots/tmr/inertia.xacro" />
-    <xacro:include filename="$(find franka_description)/robots/tmr/lidar.xacro" />
+    <xacro:include filename="$(find franka_description)/robots/tmr_v02/argo_drive.xacro" />
+    <xacro:include filename="$(find franka_description)/robots/tmr_v02/caster_wheel.xacro" />
+    <xacro:include filename="$(find franka_description)/robots/tmr_v02/rocker_arm.xacro" />
+    <xacro:include filename="$(find franka_description)/robots/tmr_v02/inertia.xacro" />
+    <xacro:include filename="$(find franka_description)/robots/tmr_v02/lidar.xacro" />
     <xacro:property name="caster_radius" value="0.03" />
     <xacro:property name="caster_x" value="0.3" />
@@ -33,5 +33,5 @@
         <origin xyz="0 0 0" rpy="0 0 ${pi}" />
         <geometry>
-          <mesh filename="package://franka_description/meshes/tmr/visual/tmr_v02.stl" />
+          <mesh filename="package://franka_description/meshes/tmr_v02/visual/tmr_v02.stl" />
         </geometry>
         <material name="white">
@@ -42,5 +42,5 @@
         <origin xyz="0 0 0" rpy="0 0 ${pi}" />
         <geometry>
-          <mesh filename="package://franka_description/meshes/tmr/collision/tmr_v02.stl" />
+          <mesh filename="package://franka_description/meshes/tmr_v02/collision/tmr_v02.stl" />
         </geometry>
       </collision>
@@ -95,6 +95,6 @@
     </xacro:lidar>
     <xacro:if value="${ros2_control}">
-      <xacro:include filename="$(find franka_description)/robots/tmr/tmr.ros2_control.xacro" />
-      <xacro:tmr_ros2_control
+      <xacro:include filename="$(find franka_description)/robots/tmr_v02/tmr_v02.ros2_control.xacro" />
+      <xacro:tmr_v02_ros2_control
         mobile_robot_id="${mobile_robot_id}"
         robot_ip="${robot_ip}"
