Commit message: feat: namespaces enabled for gazebo

File: robots/common/franka_arm.ros2_control.xacro (robot description, xacro)
@@ -9,5 +9,6 @@
                  hand:=false
                  gazebo_effort:=false
-                 arm_prefix:=''">
+                 arm_prefix:=''
+                 robot_namespace:=''">
     <xacro:property name="arm_prefix_modified" value="${'' if arm_prefix == '' else arm_prefix + '_'}" />
     <ros2_control name="${arm_prefix_modified}FrankaHardwareInterface" type="system">
@@ -88,6 +89,13 @@
     <xacro:if value="${gazebo}">
       <gazebo>
-        <plugin filename="franka_ign_ros2_control-system" name="ign_ros2_control::IgnitionROS2ControlPlugin">
-          <parameters>$(find franka_gazebo_bringup)/config/franka_gazebo_controllers.yaml</parameters>
+        <plugin
+          filename="franka_ign_ros2_control-system"
+          name="ign_ros2_control::IgnitionROS2ControlPlugin">
+          <ros>
+            <namespace>${robot_namespace}</namespace>
+          </ros>
+          <parameters>
+            $(find franka_gazebo_bringup)/config/franka_gazebo_controllers.yaml
+          </parameters>
         </plugin>
       </gazebo>

File: robots/common/franka_robot.xacro (robot description, xacro)
@@ -29,5 +29,6 @@
                       arm_prefix:=''
                       description_pkg:='franka_description'
-                      connected_to:='base'">
+                      connected_to:='base'
+                      robot_namespace:=''">
     <xacro:include filename="$(find franka_description)/robots/common/utils.xacro" />
     <xacro:include filename="$(find franka_description)/robots/common/franka_arm.xacro" />
@@ -152,4 +153,5 @@
           gazebo_effort="${gazebo_effort}"
           arm_prefix="${arm_prefix}"
+          robot_namespace="${robot_namespace}"
       />
     </xacro:if>

File: robots/fer/fer.urdf.xacro (robot description, xacro)
@@ -41,4 +41,8 @@
   <!-- Name of the description package -->
   <xacro:arg name="description_pkg" default="franka_description" />
+  <!-- The name of the frame to which the robot is connected. -->
+  <xacro:arg name="connected_to" default="base" />
+  <!-- Robot namespace -->
+  <xacro:arg name="robot_namespace" default="" />
   <!-- Append an underscore to the user-provided prefix, if non-empty. -->
   <xacro:property name="prefix" value="$(arg arm_prefix)"/>
@@ -67,5 +71,5 @@
                       arm_prefix="${modified_prefix}"
                       description_pkg="$(arg description_pkg)"
-                      connected_to= "base">
-  </xacro:franka_robot>
+                      connected_to="$(arg connected_to)"
+                      robot_namespace="$(arg robot_namespace)"/>
 </robot>

File: robots/fp3/fp3.urdf.xacro (robot description, xacro)
@@ -41,4 +41,8 @@
   <!-- Name of the description package -->
   <xacro:arg name="description_pkg" default="franka_description" />
+  <!-- The name of the frame to which the robot is connected. -->
+  <xacro:arg name="connected_to" default="base" />
+  <!-- Robot namespace -->
+   <xacro:arg name="robot_namespace" default="" />
   <!-- Append an underscore to the user-provided prefix, if non-empty. -->
   <xacro:property name="prefix" value="$(arg arm_prefix)"/>
@@ -68,5 +72,5 @@
                       arm_prefix="${modified_prefix}"
                       description_pkg="$(arg description_pkg)"
-                      connected_to= "base">
-  </xacro:franka_robot>
+                      connected_to="$(arg connected_to)"
+                      robot_namespace="$(arg robot_namespace)"/>
 </robot>

File: robots/fr3/fr3.urdf.xacro (robot description, xacro)
@@ -41,4 +41,8 @@
   <!-- Name of the description package -->
   <xacro:arg name="description_pkg" default="franka_description" />
+  <!-- The name of the frame to which the robot is connected. -->
+  <xacro:arg name="connected_to" default="base" />
+  <!-- Robot namespace -->
+  <xacro:arg name="robot_namespace" default="" />
   <!-- Append an underscore to the user-provided prefix, if non-empty. -->
   <xacro:property name="prefix" value="$(arg arm_prefix)"/>
@@ -68,5 +72,6 @@
                       arm_prefix="${modified_prefix}"
                       description_pkg="$(arg description_pkg)"
-                      connected_to= "base">
+                      connected_to="$(arg connected_to)"
+                      robot_namespace="$(arg robot_namespace)"/>
   </xacro:franka_robot>
 </robot>

File: robots/fr3_duo/fr3_duo.urdf.xacro (robot description, xacro)
@@ -42,4 +42,6 @@
   <!-- Name of the description package -->
   <xacro:arg name="description_pkg" default="franka_description" />
+  <!-- The name of the frame to which the robot is connected. -->
+  <xacro:arg name="connected_to" default="base" />
   <link name="base">
   </link>
@@ -96,5 +98,6 @@
                           arm_prefix= "${modified_prefix}"
                           description_pkg="$(arg description_pkg)"
-                          connected_to="${arm_prefixes_list[i]}_base">
+                          connected_to="${arm_prefixes_list[i]}_base"
+                          robot_namespace="">
       </xacro:franka_robot>
       <xacro:loop i="${i+1}"/>

File: robots/fr3v2/fr3v2.urdf.xacro (robot description, xacro)
@@ -41,4 +41,8 @@
   <!-- Name of the description package -->
   <xacro:arg name="description_pkg" default="franka_description" />
+  <!-- The name of the frame to which the robot is connected. -->
+  <xacro:arg name="connected_to" default="base" />
+  <!-- Robot namespace -->
+  <xacro:arg name="robot_namespace" default="" />
   <!-- Append an underscore to the user-provided prefix, if non-empty. -->
   <xacro:property name="prefix" value="$(arg arm_prefix)"/>
@@ -68,5 +72,5 @@
                       arm_prefix="${modified_prefix}"
                       description_pkg="$(arg description_pkg)"
-                      connected_to= "base">
-  </xacro:franka_robot>
+                      connected_to="$(arg connected_to)"
+                      robot_namespace="$(arg robot_namespace)"/>
 </robot>

File: robots/fr3v2_1/fr3v2_1.urdf.xacro (robot description, xacro)
@@ -41,4 +41,8 @@
   <!-- Name of the description package -->
   <xacro:arg name="description_pkg" default="franka_description" />
+  <!-- The name of the frame to which the robot is connected. -->
+  <xacro:arg name="connected_to" default="base" />
+  <!-- Robot namespace -->
+   <xacro:arg name="robot_namespace" default="" />
   <!-- Append an underscore to the user-provided prefix, if non-empty. -->
   <xacro:property name="prefix" value="$(arg arm_prefix)"/>
@@ -68,5 +72,5 @@
                       arm_prefix="${modified_prefix}"
                       description_pkg="$(arg description_pkg)"
-                      connected_to= "base">
-  </xacro:franka_robot>
+                      connected_to="$(arg connected_to)"
+                      robot_namespace="$(arg robot_namespace)"/>
 </robot>

File: robots/mobile_fr3_duo_v0_2/mobile_fr3_duo_v0_2.urdf.xacro (robot description, xacro)
@@ -43,8 +43,18 @@
   <!-- Name of the description package -->
   <xacro:arg name="description_pkg" default="franka_description" />
+  <!-- The name of the frame to which the robot is connected. -->
+  <xacro:arg name="connected_to" default="base" />
   <!-- Should the reduced tmr kinematic version (without caster wheels) be used? -->
   <xacro:arg name="reduced_version" default="false" />
-  <link name="base">
-  </link>
+  <!-- Should the arms be used? -->
+  <xacro:arg name="use_arms" default="true" />
+  <xacro:unless value="$(arg gazebo)">
+      <link name="base"/>
+      <joint name="base_joint" type="fixed">
+        <parent link="base"/>
+        <child link="base_link"/>
+        <origin rpy="0 0 0" xyz="0 0 0"/>
+      </joint>
+  </xacro:unless>
   <xacro:property name="number_of_robots" value = "3"/>
   <xacro:property name="arm_prefixes_list" value="${['','left','right']}" />
@@ -59,9 +69,4 @@
                 fake_sensor_commands="$(arg fake_sensor_commands)"
                 reduced_version="$(arg reduced_version)"/>
-        <joint name="base_joint" type="fixed">
-          <parent link="base" />
-          <child link="base_link" />
-          <origin xyz="0 0 0" rpy="0 0 0" />
-        </joint>
         <link name="franka_spine">
           <visual name="franka_spine_visual">
@@ -109,49 +114,52 @@
       </xacro:if>
       <xacro:unless value="${robot_type_i == 'tmrv0_2'}">
-        <xacro:property name="mount_to_base" value="${xacro.load_yaml('$(arg mount_kinematics)')}"/>
-        <xacro:property name="robot_prefix" value="${arm_prefixes_list[i]}"/>
-        <xacro:property name="modified_prefix" value="${robot_prefix + '_' if robot_prefix else ''}"/>
-        <joint name="${arm_prefixes_list[i]}_base_joint" type="fixed">
-          <parent link="mount_link"/>
-          <child link="${arm_prefixes_list[i]}_base"/>
-          <xacro:if value="${robot_prefix == 'left'}">
-            <xacro:property name="mount_corner" value="${mount_to_base['left']}" lazy_eval="false" />
-          </xacro:if>
-          <xacro:if value="${robot_prefix == 'right'}">
-            <xacro:property name="mount_corner" value="${mount_to_base['right']}" lazy_eval="false" />
-          </xacro:if>
-          <origin rpy="${mount_corner.kinematic.roll} ${mount_corner.kinematic.pitch} ${mount_corner.kinematic.yaw}" xyz="${mount_corner.kinematic.x} ${mount_corner.kinematic.y} ${mount_corner.kinematic.z}"/>
-        </joint>
-        <xacro:arg name="inertials_path" default="$(find franka_description)/robots/${robot_type_i}/inertials.yaml"/>
-        <xacro:arg name="kinematics_path" default="$(find franka_description)/robots/${robot_type_i}/kinematics.yaml"/>
-        <xacro:arg name="dynamics_path" default="$(find franka_description)/robots/${robot_type_i}/dynamics.yaml"/>
-        <xacro:arg name="joint_limits_path" default="$(find franka_description)/robots/${robot_type_i}/joint_limits.yaml"/>
-        <xacro:arg name="accelerometers_path" default="$(find franka_description)/robots/${robot_type_i}/accelerometers.yaml"/>
-        <xacro:franka_robot robot_type="${robot_type_i}"
-                            joint_limits="${xacro.load_yaml('$(arg joint_limits_path)')}"
-                            inertials="${xacro.load_yaml('$(arg inertials_path)')}"
-                            kinematics="${xacro.load_yaml('$(arg kinematics_path)')}"
-                            dynamics="${xacro.load_yaml('$(arg dynamics_path)')}"
-                            accelerometer_config="${xacro.load_yaml('$(arg accelerometers_path)')}"
-                            gazebo="$(arg gazebo)"
-                            hand="$(arg hand)"
-                            ee_id="$(arg ee_id)"
-                            special_connection="$(arg special_connection)"
-                            xyz_ee="$(arg xyz_ee)"
-                            rpy_ee="$(arg rpy_ee)"
-                            tcp_xyz="$(arg tcp_xyz)"
-                            tcp_rpy="$(arg tcp_rpy)"
-                            safety_distance="$(arg safety_distance)"
-                            with_sc="$(arg with_sc)"
-                            ros2_control="$(arg ros2_control)"
-                            robot_ip="${robot_ips_list[i]}"
-                            use_fake_hardware="$(arg use_fake_hardware)"
-                            fake_sensor_commands="$(arg fake_sensor_commands)"
-                            gazebo_effort="$(arg gazebo_effort)"
-                            no_prefix="$(arg no_prefix)"
-                            arm_prefix= "${modified_prefix}"
-                            description_pkg="$(arg description_pkg)"
-                            connected_to="${arm_prefixes_list[i]}_base">
-        </xacro:franka_robot>
+        <xacro:if value="$(arg use_arms)">
+          <xacro:property name="mount_to_base" value="${xacro.load_yaml('$(arg mount_kinematics)')}"/>
+          <xacro:property name="robot_prefix" value="${arm_prefixes_list[i]}"/>
+          <xacro:property name="modified_prefix" value="${robot_prefix + '_' if robot_prefix else ''}"/>
+          <joint name="${arm_prefixes_list[i]}_base_joint" type="fixed">
+            <parent link="mount_link"/>
+            <child link="${arm_prefixes_list[i]}_base"/>
+            <xacro:if value="${robot_prefix == 'left'}">
+              <xacro:property name="mount_corner" value="${mount_to_base['left']}" lazy_eval="false" />
+            </xacro:if>
+            <xacro:if value="${robot_prefix == 'right'}">
+              <xacro:property name="mount_corner" value="${mount_to_base['right']}" lazy_eval="false" />
+            </xacro:if>
+            <origin rpy="${mount_corner.kinematic.roll} ${mount_corner.kinematic.pitch} ${mount_corner.kinematic.yaw}" xyz="${mount_corner.kinematic.x} ${mount_corner.kinematic.y} ${mount_corner.kinematic.z}"/>
+          </joint>
+          <xacro:arg name="inertials_path" default="$(find franka_description)/robots/${robot_type_i}/inertials.yaml"/>
+          <xacro:arg name="kinematics_path" default="$(find franka_description)/robots/${robot_type_i}/kinematics.yaml"/>
+          <xacro:arg name="dynamics_path" default="$(find franka_description)/robots/${robot_type_i}/dynamics.yaml"/>
+          <xacro:arg name="joint_limits_path" default="$(find franka_description)/robots/${robot_type_i}/joint_limits.yaml"/>
+          <xacro:arg name="accelerometers_path" default="$(find franka_description)/robots/${robot_type_i}/accelerometers.yaml"/>
+          <xacro:franka_robot robot_type="${robot_type_i}"
+                              joint_limits="${xacro.load_yaml('$(arg joint_limits_path)')}"
+                              inertials="${xacro.load_yaml('$(arg inertials_path)')}"
+                              kinematics="${xacro.load_yaml('$(arg kinematics_path)')}"
+                              dynamics="${xacro.load_yaml('$(arg dynamics_path)')}"
+                              accelerometer_config="${xacro.load_yaml('$(arg accelerometers_path)')}"
+                              gazebo="$(arg gazebo)"
+                              hand="$(arg hand)"
+                              ee_id="$(arg ee_id)"
+                              special_connection="$(arg special_connection)"
+                              xyz_ee="$(arg xyz_ee)"
+                              rpy_ee="$(arg rpy_ee)"
+                              tcp_xyz="$(arg tcp_xyz)"
+                              tcp_rpy="$(arg tcp_rpy)"
+                              safety_distance="$(arg safety_distance)"
+                              with_sc="$(arg with_sc)"
+                              ros2_control="$(arg ros2_control)"
+                              robot_ip="${robot_ips_list[i]}"
+                              use_fake_hardware="$(arg use_fake_hardware)"
+                              fake_sensor_commands="$(arg fake_sensor_commands)"
+                              gazebo_effort="$(arg gazebo_effort)"
+                              no_prefix="$(arg no_prefix)"
+                              arm_prefix= "${modified_prefix}"
+                              description_pkg="$(arg description_pkg)"
+                              connected_to="${arm_prefixes_list[i]}_base"
+                              robot_namespace="">
+          </xacro:franka_robot>
+        </xacro:if>
       </xacro:unless>
       <xacro:loop i="${i+1}"/>

File: robots/tmrv0_2/argo_drive.xacro (robot description, xacro)
@@ -49,5 +49,13 @@
       <child  link="${name}_fixed_link" />
     </joint>
-    <link name="${name}_steering_link" />
+    <link name="${name}_steering_link">
+     <inertial>
+        <origin xyz="0 0 0" rpy="0 0 0"/>
+        <mass value="0.01"/>
+        <inertia ixx="0.0001" ixy="0.0" ixz="0.0"
+                 iyy="0.0001" iyz="0.0"
+                 izz="0.0001"/>
+      </inertial>
+    </link>
     <joint name="${mobile_robot_type}_joint_${steering_joint}" type="continuous">
       <origin xyz="0 0 0"/>

File: robots/tmrv0_2/caster_wheel.xacro (robot description, xacro)
@@ -40,5 +40,13 @@
       <child  link="${name}_fixed_link" />
     </joint>
-    <link name="${name}_steering_link" />
+    <link name="${name}_steering_link">
+      <inertial>
+          <origin xyz="0 0 0" rpy="0 0 0"/>
+          <mass value="0.01"/>
+          <inertia ixx="0.0001" ixy="0.0" ixz="0.0"
+                   iyy="0.0001" iyz="0.0"
+                   izz="0.0001"/>
+      </inertial>
+    </link>
     <joint name="${name}_steering_joint" type="continuous">
       <origin xyz="0 0 0"/>
@@ -65,4 +73,11 @@
         <xacro:caster_wheel_geometry/>
       </collision>
+      <inertial>
+        <origin xyz="0 0 0" rpy="0 0 0"/>
+        <mass value="0.001"/>
+        <inertia ixx="0.0001" ixy="0.0" ixz="0.0"
+                 iyy="0.0001" iyz="0.0"
+                 izz="0.0001"/>
+      </inertial>
     </link>
     <joint name="${name}_joint" type="continuous">

File: robots/tmrv0_2/tmrv0_2.ros2_control.xacro (robot description, xacro)
@@ -5,5 +5,7 @@
             robot_ip
             use_fake_hardware
-            fake_sensor_commands">
+            fake_sensor_commands
+            gazebo
+            robot_namespace">
     <ros2_control name="TmrHardware" type="system">
       <hardware>
@@ -16,5 +18,8 @@
           <param name="state_following_offset">0.0</param>
         </xacro:if>
-        <xacro:if value="${use_fake_hardware == 0}">
+        <xacro:if value="${gazebo}">
+          <plugin>franka_ign_ros2_control/IgnitionSystem</plugin>
+        </xacro:if>
+        <xacro:if value="${use_fake_hardware == 0 and gazebo == 0}">
           <plugin>franka_hardware/FrankaHardwareInterface</plugin>
           <param name="robot_ip">${robot_ip}</param>
@@ -55,4 +60,18 @@
       <xacro:general_purpose_io prefix="wz" command_interface="cartesian_velocity" index="5"/>
     </ros2_control>
+    <xacro:if value="${gazebo}">
+      <gazebo>
+        <plugin
+          filename="franka_ign_ros2_control-system"
+          name="ign_ros2_control::IgnitionROS2ControlPlugin">
+          <ros>
+            <namespace>${robot_namespace}</namespace>
+          </ros>
+          <parameters>
+            $(find franka_gazebo_bringup)/config/franka_gazebo_controllers.yaml
+          </parameters>
+        </plugin>
+      </gazebo>
+    </xacro:if>
   </xacro:macro>
 </robot>

File: robots/tmrv0_2/tmrv0_2.urdf.xacro (robot description, xacro)
@@ -15,8 +15,17 @@
   <!-- Should the reduced kinematic version (without caster wheels) be used? -->
   <xacro:arg name="reduced_version" default="false" />
-  <link name="base">
-  </link>
+  <!-- Should the robot be spawned in Gazebo?" -->
+  <xacro:arg name="gazebo" default="false" />
+  <!-- The namespace of the robot -->
+  <xacro:arg name="robot_namespace" default="" />
+  <xacro:unless value="$(arg gazebo)">
+      <xacro:property name="fixed_link_name" value="base"/>
+  </xacro:unless>
+  <xacro:if value="$(arg gazebo)">
+      <xacro:property name="fixed_link_name" value="world"/>
+  </xacro:if>
+  <link name="${fixed_link_name}"/>
   <joint name="base_joint" type="fixed">
-    <parent link="base"/>
+    <parent link="${fixed_link_name}"/>
     <child link="base_link"/>
     <origin rpy="0 0 0" xyz="0 0 0"/>
@@ -27,4 +36,6 @@
               use_fake_hardware="$(arg use_fake_hardware)"
               fake_sensor_commands="$(arg fake_sensor_commands)"
-              reduced_version="$(arg reduced_version)"/>
+              reduced_version="$(arg reduced_version)"
+              robot_namespace="$(arg robot_namespace)"
+              gazebo="$(arg gazebo)"/>
 </robot>

File: robots/tmrv0_2/tmrv0_2.xacro (robot description, xacro)
@@ -7,5 +7,7 @@
                   use_fake_hardware:=false
                   fake_sensor_commands:=false
-                  reduced_version:=false">
+                  reduced_version:=false
+                  robot_namespace:=''
+                  gazebo:=false">
     <xacro:include filename="$(find franka_description)/robots/tmrv0_2/argo_drive.xacro" />
     <xacro:include filename="$(find franka_description)/robots/tmrv0_2/caster_wheel.xacro" />
@@ -139,4 +141,6 @@
         use_fake_hardware="${use_fake_hardware}"
         fake_sensor_commands="${fake_sensor_commands}"
+        robot_namespace="${robot_namespace}"
+        gazebo="${gazebo}"
       />
     </xacro:if>

Commit message: fix: properly handle arm_prefixes in srdf

File: robots/common/franka_arm.ros2_control.xacro (robot description, xacro)
@@ -11,6 +11,5 @@
                  arm_prefix:=''
                  robot_namespace:=''">
-    <xacro:property name="arm_prefix_modified" value="${'' if arm_prefix == '' else arm_prefix + '_'}" />
-    <ros2_control name="${arm_prefix_modified}FrankaHardwareInterface" type="system">
+    <ros2_control name="${arm_prefix}FrankaHardwareInterface" type="system">
         <hardware>
           <param name="version">0.1.0</param>
@@ -63,5 +62,5 @@
       </xacro:if>
       <xacro:macro name="general_purpose_io" params="prefix command_interface index">
-        <gpio name="${prefix}">
+        <gpio name="${arm_prefix}${prefix}">
           <command_interface name="${command_interface}"/>
           <param name="index">${index}</param>

File: robots/fer/fer.srdf.xacro (robot description, xacro)
@@ -12,9 +12,12 @@
   <!-- Which end-effector would be mounted at the flange?" -->
   <xacro:arg name="ee_id" default="franka_hand" />
+  <!-- Append an underscore to the user-provided prefix, if non-empty. -->
+  <xacro:property name="prefix" value="$(arg arm_prefix)"/>
+  <xacro:property name="modified_prefix" value="${prefix + '_' if prefix else ''}"/>
   <xacro:franka_arm_srdf robot_type="$(arg robot_type)"
                       hand="$(arg hand)"
                       ee_id="$(arg ee_id)"
                       no_prefix="$(arg no_prefix)"
-                      arm_prefix= "$(arg arm_prefix)">
+                      arm_prefix="$(modified_prefix)">
   </xacro:franka_arm_srdf>
 </robot>
