Commit message: fix: passive state interfaces added for gazebo

File: robots/common/franka_robot.xacro (robot description, xacro)
@@ -97,15 +97,4 @@
     <!-- Definition of additional Gazebo tags -->
     <xacro:if value="${gazebo}">
-      <xacro:if value="${parent != ''}">
-        <!-- Gazebo requires a joint to a link called "world" for statically mounted robots -->
-        <xacro:if value="${parent == 'world'}">
-          <link name="${parent}" />
-        </xacro:if>
-        <joint name="${parent}_joint" type="fixed">
-          <origin xyz="${xyz}" rpy="${rpy}" />
-          <parent link="${parent}" />
-          <child  link="${arm_prefix}${robot_type}_link0" />
-        </joint>
-      </xacro:if>
       <xacro:gazebo-joint joint="${arm_prefix}${robot_type}_joint1" transmission="hardware_interface/PositionJointInterface" />
       <xacro:gazebo-joint joint="${arm_prefix}${robot_type}_joint2" transmission="hardware_interface/PositionJointInterface" />

File: robots/fer/fer.urdf.xacro (robot description, xacro)
@@ -48,4 +48,16 @@
   <xacro:property name="prefix" value="$(arg arm_prefix)"/>
   <xacro:property name="modified_prefix" value="${prefix + '_' if prefix else ''}"/>
+  <!--Position offset with respect to the world-->
+  <xacro:arg name="xyz" default="0 0 0" />
+  <!--Rotation offset with respect to the world-->
+  <xacro:arg name="rpy" default="0 0 0" />
+  <xacro:if value="$(arg gazebo)">
+    <link name="world" />
+    <joint name="world_joint" type="fixed">
+      <origin xyz="$(arg xyz)" rpy="$(arg rpy)" />
+      <parent link="world" />
+      <child  link="${modified_prefix}$(arg robot_type)_link0" />
+    </joint>
+  </xacro:if>
   <xacro:franka_robot robot_type="fer"
                       joint_limits="${xacro.load_yaml('$(find franka_description)/robots/fer/joint_limits.yaml')}"

File: robots/fp3/fp3.urdf.xacro (robot description, xacro)
@@ -48,4 +48,16 @@
   <xacro:property name="prefix" value="$(arg arm_prefix)"/>
   <xacro:property name="modified_prefix" value="${prefix + '_' if prefix else ''}"/>
+  <!--Position offset with respect to the world-->
+  <xacro:arg name="xyz" default="0 0 0" />
+  <!--Rotation offset with respect to the world-->
+  <xacro:arg name="rpy" default="0 0 0" />
+  <xacro:if value="$(arg gazebo)">
+    <link name="world" />
+    <joint name="world_joint" type="fixed">
+      <origin xyz="$(arg xyz)" rpy="$(arg rpy)" />
+      <parent link="world" />
+      <child  link="${modified_prefix}$(arg robot_type)_link0" />
+    </joint>
+  </xacro:if>
   <xacro:franka_robot robot_type="fp3"
                       joint_limits="${xacro.load_yaml('$(find franka_description)/robots/fp3/joint_limits.yaml')}"

File: robots/fr3/fr3.urdf.xacro (robot description, xacro)
@@ -48,4 +48,16 @@
   <xacro:property name="prefix" value="$(arg arm_prefix)"/>
   <xacro:property name="modified_prefix" value="${prefix + '_' if prefix else ''}"/>
+  <!--Position offset with respect to the world-->
+  <xacro:arg name="xyz" default="0 0 0" />
+  <!--Rotation offset with respect to the world-->
+  <xacro:arg name="rpy" default="0 0 0" />
+  <xacro:if value="$(arg gazebo)">
+    <link name="world" />
+    <joint name="world_joint" type="fixed">
+      <origin xyz="$(arg xyz)" rpy="$(arg rpy)" />
+      <parent link="world" />
+      <child  link="${modified_prefix}$(arg robot_type)_link0" />
+    </joint>
+  </xacro:if>
   <xacro:franka_robot robot_type="fr3"
                       joint_limits="${xacro.load_yaml('$(find franka_description)/robots/fr3/joint_limits.yaml')}"

File: robots/fr3v2/fr3v2.urdf.xacro (robot description, xacro)
@@ -48,4 +48,16 @@
   <xacro:property name="prefix" value="$(arg arm_prefix)"/>
   <xacro:property name="modified_prefix" value="${prefix + '_' if prefix else ''}"/>
+  <!--Position offset with respect to the world-->
+  <xacro:arg name="xyz" default="0 0 0" />
+  <!--Rotation offset with respect to the world-->
+  <xacro:arg name="rpy" default="0 0 0" />
+  <xacro:if value="$(arg gazebo)">
+    <link name="world" />
+    <joint name="world_joint" type="fixed">
+      <origin xyz="$(arg xyz)" rpy="$(arg rpy)" />
+      <parent link="world" />
+      <child  link="${modified_prefix}$(arg robot_type)_link0" />
+    </joint>
+  </xacro:if>
   <xacro:franka_robot robot_type="fr3v2"
                       joint_limits="${xacro.load_yaml('$(find franka_description)/robots/fr3v2/joint_limits.yaml')}"

File: robots/fr3v2_1/fr3v2_1.urdf.xacro (robot description, xacro)
@@ -48,4 +48,16 @@
   <xacro:property name="prefix" value="$(arg arm_prefix)"/>
   <xacro:property name="modified_prefix" value="${prefix + '_' if prefix else ''}"/>
+  <!--Position offset with respect to the world-->
+  <xacro:arg name="xyz" default="0 0 0" />
+  <!--Rotation offset with respect to the world-->
+  <xacro:arg name="rpy" default="0 0 0" />
+  <xacro:if value="$(arg gazebo)">
+    <link name="world" />
+    <joint name="world_joint" type="fixed">
+      <origin xyz="$(arg xyz)" rpy="$(arg rpy)" />
+      <parent link="world" />
+      <child  link="${modified_prefix}$(arg robot_type)_link0" />
+    </joint>
+  </xacro:if>
   <xacro:franka_robot robot_type="fr3v2_1"
                       joint_limits="${xacro.load_yaml('$(find franka_description)/robots/fr3v2_1/joint_limits.yaml')}"

File: robots/tmrv0_2/argo_drive.xacro (robot description, xacro)
@@ -7,5 +7,5 @@
     <xacro:property name="base_height" value="0.077" />
     <xacro:property name="offset_wheel" value="0.085" />
-    <xacro:property name="mass" value="0.5" />
+    <xacro:property name="mass" value="2.5" />
     <xacro:if value="${name == 'argo_drive_front'}">
       <xacro:property name="steering_joint" value="0" />
@@ -64,5 +64,5 @@
       <axis   xyz="0 0 1" />
       <limit  effort="500" velocity="20" />
-      <dynamics damping="0.003" friction="0.0"/>
+      <dynamics damping="20.0" friction="5.0"/>
     </joint>
     <link name="${name}_link" >
@@ -90,5 +90,5 @@
       <axis   xyz="0 1 0" />
       <limit  effort="500" velocity="20" />
-      <dynamics damping="0.003" friction="0.0"/>
+      <dynamics damping="5.0" friction="1.0"/>
     </joint>
   </xacro:macro>

File: robots/tmrv0_2/tmrv0_2.ros2_control.xacro (robot description, xacro)
@@ -32,4 +32,7 @@
             <param name="initial_value">0.0</param>
           </state_interface>
+          <state_interface name="velocity">
+            <param name="initial_value">0.0</param>
+          </state_interface>
         </joint>
       </xacro:macro>
@@ -37,4 +40,7 @@
         <joint name="${joint_name}">
           <command_interface name="velocity"/>
+          <state_interface name="position">
+            <param name="initial_value">0.0</param>
+          </state_interface>
           <state_interface name="velocity">
             <param name="initial_value">0.0</param>
@@ -46,4 +52,51 @@
       <xacro:configure_steering_joint joint_name="${mobile_robot_type}_joint_2"/>
       <xacro:configure_driving_joint joint_name="${mobile_robot_type}_joint_3"/>
+      <xacro:if value="${gazebo}">
+        <!-- Rocker Arm -->
+        <joint name="rocker_arm_joint">
+          <state_interface name="position">
+            <param name="initial_value">0.0</param>
+          </state_interface>
+          <state_interface name="velocity">
+            <param name="initial_value">0.0</param>
+          </state_interface>
+        </joint>
+        <!-- Front caster steering -->
+        <joint name="caster_front_left_steering_joint">
+          <state_interface name="position">
+            <param name="initial_value">0.0</param>
+          </state_interface>
+          <state_interface name="velocity">
+            <param name="initial_value">0.0</param>
+          </state_interface>
+        </joint>
+        <!-- Front caster joint -->
+        <joint name="caster_front_left_joint">
+          <state_interface name="position">
+            <param name="initial_value">0.0</param>
+          </state_interface>
+          <state_interface name="velocity">
+            <param name="initial_value">0.0</param>
+          </state_interface>
+        </joint>
+        <!-- Rear caster steering -->
+        <joint name="caster_rear_right_steering_joint">
+          <state_interface name="position">
+            <param name="initial_value">0.0</param>
+          </state_interface>
+          <state_interface name="velocity">
+            <param name="initial_value">0.0</param>
+          </state_interface>
+        </joint>
+        <!-- Rear caster joint -->
+        <joint name="caster_rear_right_joint">
+          <state_interface name="position">
+            <param name="initial_value">0.0</param>
+          </state_interface>
+          <state_interface name="velocity">
+            <param name="initial_value">0.0</param>
+          </state_interface>
+        </joint>
+      </xacro:if>
       <xacro:macro name="general_purpose_io" params="prefix command_interface index">
         <gpio name="${prefix}">

File: robots/tmrv0_2/tmrv0_2.urdf.xacro (robot description, xacro)
@@ -20,15 +20,11 @@
   <xacro:arg name="robot_namespace" default="" />
   <xacro:unless value="$(arg gazebo)">
-      <xacro:property name="fixed_link_name" value="base"/>
+    <link name="base"/>
+    <joint name="base_joint" type="fixed">
+      <parent link="base"/>
+      <child link="base_link"/>
+      <origin rpy="0 0 0" xyz="0 0 0"/>
+    </joint>
   </xacro:unless>
-  <xacro:if value="$(arg gazebo)">
-      <xacro:property name="fixed_link_name" value="world"/>
-  </xacro:if>
-  <link name="${fixed_link_name}"/>
-  <joint name="base_joint" type="fixed">
-    <parent link="${fixed_link_name}"/>
-    <child link="base_link"/>
-    <origin rpy="0 0 0" xyz="0 0 0"/>
-  </joint>
   <xacro:tmrv0_2 mobile_robot_type="$(arg robot_type)"
               robot_ip="$(arg robot_ip)"

File: robots/tmrv0_2/tmrv0_2.xacro (robot description, xacro)
@@ -113,5 +113,5 @@
       <parent link="base_link" />
       <child link="right_mounting_point" />
-      <origin xyz="0.0 0.272712 0.1145" rpy="${pi} 0 ${pi/2}" />
+      <origin xyz="0.0 -0.272712 0.1145" rpy="${pi} 0 -${pi/2}" />
     </joint>
     <link name="left_mounting_point"/>
@@ -119,5 +119,5 @@
       <parent link="base_link" />
       <child link="left_mounting_point" />
-      <origin xyz="0.0 -0.272712 0.1145" rpy="${pi} 0 -${pi/2}" />
+      <origin xyz="0.0 0.272712 0.1145" rpy="${pi} 0 ${pi/2}" />
     </joint>
     <!-- Lidars -->

Commit message: add option to set the gripper to robotiq_arg85

File: robots/common/franka_robot.xacro (robot description, xacro)
@@ -68,5 +68,28 @@
       />
     </xacro:if>
-    <xacro:if value="${hand and ee_id != 'none' and ee_id != 'franka_hand'}">
+    <xacro:if value="${hand and ee_id == 'robotiq_arg85'}">
+      <xacro:include filename="$(find franka_description)/end_effectors/robotiq_arg85/robotiq_arg85.xacro"/>
+      <xacro:property name="connection"
+        value="${special_connection if special_connection != '' else robot_type + '_link8'}"/>
+      <xacro:robotiq_arg85
+        connected_to="${arm_prefix}${connection}"
+        robot_type="${robot_type}"
+        arm_prefix="${arm_prefix}"
+        ee_id="${ee_id}"
+        rpy_ee="${rpy_ee}"
+        xyz_ee="${xyz_ee}"
+        tcp_xyz="${tcp_xyz}"
+        tcp_rpy="${tcp_rpy}"
+        safety_distance="${safety_distance}"
+        gazebo="${gazebo}"
+        description_pkg="${description_pkg}"
+        with_sc="${with_sc}"
+        no_prefix="${no_prefix}"
+        ros2_control="${ros2_control}"
+        use_fake_hardware="${use_fake_hardware}"
+        mock_sensor_commands="${fake_sensor_commands}"
+      />
+    </xacro:if>
+    <xacro:if value="${hand and ee_id != 'none' and ee_id != 'franka_hand' and ee_id != 'robotiq_arg85'}">
       <xacro:include filename="$(find franka_description)/end_effectors/common/ee_with_one_link.xacro"/>
       <xacro:include filename="$(find franka_description)/end_effectors/common/utils.xacro"/>
