Commit message: fix: default the tcp offset to the mounted end effector's own value
The tcp offset is a property of the end effector, but it was specified in two
places that disagreed with it. The franka_robot macro declared tcp_xyz:='0 0 0',
while every robot entry point declared '0 0 0.1034'. The offset therefore
survived only because the entry point passed it back down, and two defects
followed from that.

Calling the franka_robot macro directly without tcp_xyz - which downstream
packages and user xacros do - silently produced hand_tcp coincident with the
mounting frame, reported as issue #31 on GitHub. Separately, the entry points
hardcoded the franka hand's 0.1034 for every end effector, so a robot built with
ee_id:=cobot_pump placed the pump tcp 1.6 mm short of the 0 0 0.105 the pump
itself declares.

Make an unspecified tcp_xyz resolve to the end effector's own offset, and drop
the hardcoded value from the entry points so the resolution is what decides. An
explicitly passed tcp_xyz still wins everywhere.

Add regression tests pinning the resolved offset to what the end effector
produces standalone, exercised through both the entry points and a direct macro
call, plus one asserting an explicit override still takes precedence. All three
fail before this change.

Verified by generating every robot, end effector, self-collision, prefix and
override combination (50 descriptions) before and after: output is
byte-identical except for the ten cobot pump variants, which gain the corrected
offset. check_urdf passes on all of them.

Reported in https://github.com/frankarobotics/franka_description/issues/31

Signed-off-by: Kamal Mohy El Dine <kamal.mohy@franka.de>

File: robots/common/franka_robot.xacro (robot description, xacro)
@@ -8,5 +8,5 @@
                       xyz_ee:='0 0 0'
                       rpy_ee:='0 0 0'
-                      tcp_xyz:='0 0 0'
+                      tcp_xyz:=''
                       tcp_rpy:='0 0 0'
                       safety_distance:='0.03'
@@ -22,4 +22,11 @@
     <xacro:include filename="$(find franka_description)/robots/common/utils.xacro"/>
     <xacro:include filename="$(find franka_description)/robots/common/franka_arm.xacro"/>
+    <!-- The tcp offset belongs to the end effector, so an empty tcp_xyz resolves to
+         that end effector's own value rather than to zero. These must match the
+         defaults in end_effectors/<ee_id>/<ee_id>_arguments.xacro, which
+         test_tcp_offset_matches_end_effector enforces. -->
+    <xacro:property name="ee_tcp_xyz"
+      value="${'0 0 0.1034' if ee_id == 'franka_hand' else '0 0 0.105' if ee_id == 'cobot_pump' else '0 0 0'}"/>
+    <xacro:property name="tcp_xyz_resolved" value="${ee_tcp_xyz if tcp_xyz == '' else tcp_xyz}"/>
     <xacro:franka_arm
       robot_type="${robot_type}"
@@ -53,5 +60,5 @@
         rpy_ee="${rpy_ee}"
         xyz_ee="${xyz_ee}"
-        tcp_xyz="${tcp_xyz}"
+        tcp_xyz="${tcp_xyz_resolved}"
         tcp_rpy="${tcp_rpy}"
         safety_distance="${safety_distance}"
@@ -74,5 +81,5 @@
         rpy_ee="${rpy_ee}"
         xyz_ee="${xyz_ee}"
-        tcp_xyz="${tcp_xyz}"
+        tcp_xyz="${tcp_xyz_resolved}"
         tcp_rpy="${tcp_rpy}"
         safety_distance="${safety_distance}"

File: robots/fer/fer.urdf.xacro (robot description, xacro)
@@ -20,5 +20,5 @@
   <xacro:arg name="rpy_ee" default="0 0 ${-pi/4}"/>
   <!-- Position offset between ee frame and tcp frame -->
-  <xacro:arg name="tcp_xyz" default="0 0 0.1034"/>
+  <xacro:arg name="tcp_xyz" default=""/>
   <!-- Rotation offset between ee frame and tcp frame -->
   <xacro:arg name="tcp_rpy" default="0 0 0"/>

File: robots/fp3/fp3.urdf.xacro (robot description, xacro)
@@ -20,5 +20,5 @@
   <xacro:arg name="rpy_ee" default="0 0 ${-pi/4}"/>
   <!-- Position offset between ee frame and tcp frame -->
-  <xacro:arg name="tcp_xyz" default="0 0 0.1034"/>
+  <xacro:arg name="tcp_xyz" default=""/>
   <!-- Rotation offset between ee frame and tcp frame -->
   <xacro:arg name="tcp_rpy" default="0 0 0"/>

File: robots/fr3/fr3.urdf.xacro (robot description, xacro)
@@ -20,5 +20,5 @@
   <xacro:arg name="rpy_ee" default="0 0 ${-pi/4}"/>
   <!-- Position offset between ee frame and tcp frame -->
-  <xacro:arg name="tcp_xyz" default="0 0 0.1034"/>
+  <xacro:arg name="tcp_xyz" default=""/>
   <!-- Rotation offset between ee frame and tcp frame -->
   <xacro:arg name="tcp_rpy" default="0 0 0"/>

File: robots/fr3_duo/fr3_duo.urdf.xacro (robot description, xacro)
@@ -19,5 +19,5 @@
   <xacro:arg name="rpy_ee" default="0 0 ${-pi/4}"/>
   <!-- Position offset between ee frame and tcp frame -->
-  <xacro:arg name="tcp_xyz" default="0 0 0.1034"/>
+  <xacro:arg name="tcp_xyz" default=""/>
   <!-- Rotation offset between ee frame and tcp frame -->
   <xacro:arg name="tcp_rpy" default="0 0 0"/>

File: robots/fr3v2/fr3v2.urdf.xacro (robot description, xacro)
@@ -20,5 +20,5 @@
   <xacro:arg name="rpy_ee" default="0 0 ${-pi/4}"/>
   <!-- Position offset between ee frame and tcp frame -->
-  <xacro:arg name="tcp_xyz" default="0 0 0.1034"/>
+  <xacro:arg name="tcp_xyz" default=""/>
   <!-- Rotation offset between ee frame and tcp frame -->
   <xacro:arg name="tcp_rpy" default="0 0 0"/>

File: robots/fr3v2_1/fr3v2_1.urdf.xacro (robot description, xacro)
@@ -20,5 +20,5 @@
   <xacro:arg name="rpy_ee" default="0 0 ${-pi/4}"/>
   <!-- Position offset between ee frame and tcp frame -->
-  <xacro:arg name="tcp_xyz" default="0 0 0.1034"/>
+  <xacro:arg name="tcp_xyz" default=""/>
   <!-- Rotation offset between ee frame and tcp frame -->
   <xacro:arg name="tcp_rpy" default="0 0 0"/>

File: robots/mobile_fr3_duo_v0_2/mobile_fr3_duo_v0_2.urdf.xacro (robot description, xacro)
@@ -19,5 +19,5 @@
   <xacro:arg name="rpy_ee" default="0 0 ${-pi/4}"/>
   <!-- Position offset between ee frame and tcp frame -->
-  <xacro:arg name="tcp_xyz" default="0 0 0.1034"/>
+  <xacro:arg name="tcp_xyz" default=""/>
   <!-- Rotation offset between ee frame and tcp frame -->
   <xacro:arg name="tcp_rpy" default="0 0 0"/>
