Commit message: fix: tip the MoveIt planning chain at the cobot pump's tcp
The arm group's chain tipped at hand_tcp for the franka hand and at link8 for
everything else, so the two supported end effectors disagreed about what a pose
goal means. With a pump mounted, a goal named the flange while the pump's own
tcp frame, 105 mm further along z, was present in the URDF but unreachable as a
planning target. Planning to the tool is the reason that frame exists.

Resolve the tip from the mounted end effector instead, keeping the flange for
ids that declare no tcp of their own and for hand:=false, so no unknown ee_id
can name a link the URDF lacks.

Add regression tests pinning the chain tip to the tcp link the URDF places for
the mounted end effector, and pinning the flange when nothing is mounted. The
first fails on the ten cobot pump variants before this change.

Verified by generating every arm, end effector, prefix and hand combination (61
SRDFs) before and after: byte-identical except the ten cobot pump variants that
carry a hand, whose only changed line is the chain tip. Loading the result
through MoveIt's own parser gives a valid seven joint chain whose ready-pose tip
sits 105 mm below the previous one.

MIGRATION: pose goals for ee_id:=cobot_pump shift by 105 mm along the flange z
axis. Setups that added that offset themselves must drop it.

Signed-off-by: Kamal Mohy El Dine <kamal.mohy@franka.de>

File: robots/common/franka_arm.srdf.xacro (robot description, xacro)
@@ -4,5 +4,7 @@
         <xacro:property name="prefix" value="${'' if no_prefix else arm_prefix + robot_type + '_'}" />
         <xacro:include filename="$(find franka_description)/robots/common/group_definition.xacro"/>
-        <xacro:property name="tip_link" value="${prefix + 'hand_tcp' if hand and ee_id == 'franka_hand' else prefix + 'link8'}"/>
+        <xacro:property name="ee_tcp_link"
+            value="${'hand_tcp' if ee_id == 'franka_hand' else 'cobot_pump_tcp' if ee_id == 'cobot_pump' else 'link8'}"/>
+        <xacro:property name="tip_link" value="${prefix + ee_tcp_link if hand else prefix + 'link8'}"/>
         <xacro:group_definition prefix="${prefix}" group_name="${prefix}arm" tip_link="${tip_link}"/>
         <virtual_joint name="virtual_joint" type="fixed" parent_frame="world" child_link="base"/>
