Commit message: refactor: Remove gazebo tags/macros/args from franka_description
Make the description package simulator-agnostic. All gazebo SDF and
transmission machinery, the gazebo world anchor, and the gazebo-specific
self-collision suppression are removed; the gazebo:=false argument and the
gazebo_ros export are dropped throughout robots, end_effectors and the URDF
generation workflow.

Self-collision geometry is now gated by the include_self_collision_geometry
capability flag instead of a gazebo toggle. The removed gazebo content is
relocated to franka_gazebo, which owns the simulator-specific blocks.

The removal of the public gazebo xacro argument is recorded in a CHANGELOG
UNRELEASED migration note: consumers that passed gazebo:=true must now use
the franka_gazebo bringup entry points; the old argument is inert.

Behavior-preserving: URDF expansions are byte-identical to before.

File: end_effectors/cobot_pump/cobot_pump.urdf.xacro (robot description, xacro)
@@ -13,5 +13,5 @@
                           tcp_rpy="$(arg tcp_rpy)"
                           safety_distance="$(arg safety_distance)"
-                          gazebo="$(arg gazebo)"
+                          include_self_collision_geometry="$(arg include_self_collision_geometry)"
                           description_pkg="$(arg description_pkg)"
                           with_sc="$(arg with_sc)">

File: end_effectors/cobot_pump/cobot_pump_arguments.xacro (robot description, xacro)
@@ -19,6 +19,6 @@
   <!-- Safety distance for the collision capsules -->
   <xacro:arg name="safety_distance" default="0.03" />
-  <!-- Is the robot being simulated in gazebo? -->
-  <xacro:arg name="gazebo" default="false" />
+  <!-- Emit the coarse self-collision capsule geometry inside the *_sc sub-links? -->
+  <xacro:arg name="include_self_collision_geometry" default="true" />
   <!-- Name of the description package -->
   <xacro:arg name="description_pkg" default="franka_description" />

File: end_effectors/common/ee_with_one_link.xacro (robot description, xacro)
@@ -2,5 +2,5 @@
 <robot xmlns:xacro="http://www.ros.org/wiki/xacro" name="ee_with_one_link">
   <!-- safety_distance: Minimum safety distance in [m] by which the collision volumes are expanded and which is enforced during robot motions -->
-  <xacro:macro name="ee_with_one_link" params="connected_to:='' robot_type arm_prefix:='' ee_id ee_inertials rpy_ee:='0 0 0' xyz_ee:='0 0 0' tcp_xyz:='0 0 0' tcp_rpy:='0 0 0' safety_distance:=0 gazebo:=false description_pkg:=franka_description with_sc:=false">
+  <xacro:macro name="ee_with_one_link" params="connected_to:='' robot_type arm_prefix:='' ee_id ee_inertials rpy_ee:='0 0 0' xyz_ee:='0 0 0' tcp_xyz:='0 0 0' tcp_rpy:='0 0 0' safety_distance:=0 include_self_collision_geometry:=true description_pkg:=franka_description with_sc:=false">
     <xacro:property name="ee_prefix" default="robot_"/>
     <xacro:unless value="${robot_type == ''}">
@@ -14,5 +14,5 @@
       </joint>
     </xacro:unless>
-    <xacro:ee_link_with_sc name="${ee_id}" gazebo="${gazebo}" with_sc="${with_sc}">
+    <xacro:ee_link_with_sc name="${ee_id}" include_self_collision_geometry="${include_self_collision_geometry}" with_sc="${with_sc}">
       <self_collision_geometries>
         <xacro:collision_capsule xyz="0 0 0.04" direction="y" radius="${0.04+safety_distance}" length="0.1" />

File: end_effectors/common/franka_hand.xacro (robot description, xacro)
@@ -11,5 +11,5 @@
                        tcp_rpy:='0 0 0'
                        safety_distance:=0
-                       gazebo:=false
+                       include_self_collision_geometry:=true
                        description_pkg:=franka_description
                        with_sc:=false
@@ -26,5 +26,5 @@
       </joint>
     </xacro:unless>
-    <xacro:ee_link_with_sc name="hand" gazebo="${gazebo}" with_sc="${with_sc}">
+    <xacro:ee_link_with_sc name="hand" include_self_collision_geometry="${include_self_collision_geometry}" with_sc="${with_sc}">
       <self_collision_geometries>
         <xacro:collision_capsule xyz="0 0 0.04" direction="y" radius="${0.04+safety_distance}" length="0.1" />

File: end_effectors/franka_hand/franka_hand.urdf.xacro (robot description, xacro)
@@ -13,5 +13,5 @@
                      tcp_rpy="$(arg tcp_rpy)"
                      safety_distance="$(arg safety_distance)"
-                     gazebo="$(arg gazebo)"
+                     include_self_collision_geometry="$(arg include_self_collision_geometry)"
                      description_pkg="$(arg description_pkg)"
                      with_sc="$(arg with_sc)">

File: end_effectors/franka_hand/franka_hand_arguments.xacro (robot description, xacro)
@@ -21,6 +21,6 @@
   <!-- Safety distance for the collision capsules -->
   <xacro:arg name="safety_distance" default="0.03" />
-  <!-- Is the robot being simulated in gazebo? -->
-  <xacro:arg name="gazebo" default="false" />
+  <!-- Emit the coarse self-collision capsule geometry inside the *_sc sub-links? -->
+  <xacro:arg name="include_self_collision_geometry" default="true" />
   <!-- Name of the description package -->
   <xacro:arg name="description_pkg" default="franka_description" />

File: robots/common/franka_arm.xacro (robot description, xacro)
@@ -8,5 +8,5 @@
   <!-- inertials: description of the inertials that comes from a YAML file. Example definition: ${xacro.load_yaml('$(find franka_description)/robots/fr3/inertials.yaml')} -->
   <!-- dynamics: description of the dynamics that comes from a YAML file. Example definition: ${xacro.load_yaml('$(find franka_description)/robots/fr3/dynamics.yaml')} -->
-  <xacro:macro name="franka_arm" params="robot_type arm_prefix:='' no_prefix:=false description_pkg:='franka_description' connected_to:='base' xyz:='0 0 0' rpy:='0 0 0' gazebo:='false' safety_distance:=0 with_sc:=false" >
+  <xacro:macro name="franka_arm" params="robot_type arm_prefix:='' no_prefix:=false description_pkg:='franka_description' connected_to:='base' xyz:='0 0 0' rpy:='0 0 0' include_self_collision_geometry:='true' safety_distance:=0 with_sc:=false" >
     <xacro:property name="joint_limits" value="${xacro.load_yaml('$(find franka_description)/robots/' + robot_type + '/joint_limits.yaml')}"/>
     <xacro:property name="inertials" value="${xacro.load_yaml('$(find franka_description)/robots/' + robot_type  + '/inertials.yaml')}"/>
@@ -17,7 +17,4 @@
     <xacro:property name="prefix" value="${'' if no_prefix else arm_prefix + robot_type + '_'}" />
     <xacro:property name="with_accelerometers" value="${'false' if accelerometer_config == 'none' else 'true'}" />
-    <xacro:if value="${gazebo and connected_to == 'base'}">
-      <xacro:property name="connected_to" value="" />
-    </xacro:if>
     <xacro:unless value="${not connected_to}">
       <link name="${connected_to}">
@@ -29,10 +26,10 @@
       </joint>
     </xacro:unless>
-    <xacro:link_with_sc no_prefix="${no_prefix}" name="link0" gazebo="${gazebo}" with_sc="${with_sc}" with_accelerometers="${with_accelerometers}">
+    <xacro:link_with_sc no_prefix="${no_prefix}" name="link0" include_self_collision_geometry="${include_self_collision_geometry}" with_sc="${with_sc}" with_accelerometers="${with_accelerometers}">
       <self_collision_geometries>
         <xacro:collision_capsule xyz="-0.075 0 0.06" direction="x" radius="${0.06+safety_distance}" length="0.03" />
       </self_collision_geometries>
     </xacro:link_with_sc>
-    <xacro:link_with_sc no_prefix="${no_prefix}" name="link1" gazebo="${gazebo}" with_sc="${with_sc}" with_accelerometers="${with_accelerometers}">
+    <xacro:link_with_sc no_prefix="${no_prefix}" name="link1" include_self_collision_geometry="${include_self_collision_geometry}" with_sc="${with_sc}" with_accelerometers="${with_accelerometers}">
       <self_collision_geometries>
         <xacro:collision_capsule xyz="0 0 -191.5e-3" radius="${0.06+safety_distance}" length="0.283" />
@@ -47,5 +44,5 @@
       <xacro:franka-dynamics name="joint1" config="${dynamics}" />
     </joint>
-    <xacro:link_with_sc no_prefix="${no_prefix}" name="link2" gazebo="${gazebo}" with_sc="${with_sc}" with_accelerometers="${with_accelerometers}">
+    <xacro:link_with_sc no_prefix="${no_prefix}" name="link2" include_self_collision_geometry="${include_self_collision_geometry}" with_sc="${with_sc}" with_accelerometers="${with_accelerometers}">
       <self_collision_geometries>
         <xacro:collision_capsule xyz="0 0 0" radius="${0.06+safety_distance}" length="0.12" />
@@ -60,5 +57,5 @@
       <xacro:franka-dynamics name="joint2" config="${dynamics}" />
     </joint>
-    <xacro:link_with_sc no_prefix="${no_prefix}" name="link3" gazebo="${gazebo}" with_sc="${with_sc}" with_accelerometers="${with_accelerometers}">
+    <xacro:link_with_sc no_prefix="${no_prefix}" name="link3" include_self_collision_geometry="${include_self_collision_geometry}" with_sc="${with_sc}" with_accelerometers="${with_accelerometers}">
       <self_collision_geometries>
         <xacro:collision_capsule xyz="0 0 -0.145" radius="${0.06+safety_distance}" length="0.15" />
@@ -73,5 +70,5 @@
       <xacro:franka-dynamics name="joint3" config="${dynamics}" />
     </joint>
-    <xacro:link_with_sc no_prefix="${no_prefix}" name="link4" gazebo="${gazebo}" with_sc="${with_sc}" with_accelerometers="${with_accelerometers}">
+    <xacro:link_with_sc no_prefix="${no_prefix}" name="link4" include_self_collision_geometry="${include_self_collision_geometry}" with_sc="${with_sc}" with_accelerometers="${with_accelerometers}">
       <self_collision_geometries>
         <xacro:collision_capsule xyz="0 0 0" radius="${0.06+safety_distance}" length="0.12" />
@@ -86,5 +83,5 @@
       <xacro:franka-dynamics name="joint4" config="${dynamics}" />
     </joint>
-    <xacro:link_with_sc no_prefix="${no_prefix}" name="link5" gazebo="${gazebo}" with_sc="${with_sc}" with_accelerometers="${with_accelerometers}">
+    <xacro:link_with_sc no_prefix="${no_prefix}" name="link5" include_self_collision_geometry="${include_self_collision_geometry}" with_sc="${with_sc}" with_accelerometers="${with_accelerometers}">
       <self_collision_geometries>
         <xacro:collision_capsule xyz="0 0 -0.26"    radius="${0.060+safety_distance}" length="0.10" />
@@ -100,5 +97,5 @@
       <xacro:franka-dynamics name="joint5" config="${dynamics}" />
     </joint>
-    <xacro:link_with_sc no_prefix="${no_prefix}" name="link6" gazebo="${gazebo}" with_sc="${with_sc}" with_accelerometers="false">
+    <xacro:link_with_sc no_prefix="${no_prefix}" name="link6" include_self_collision_geometry="${include_self_collision_geometry}" with_sc="${with_sc}" with_accelerometers="false">
       <self_collision_geometries>
         <xacro:collision_capsule xyz="0 0 -0.03" radius="${0.05+safety_distance}" length="0.08" />
@@ -113,5 +110,5 @@
       <xacro:franka-dynamics name="joint6" config="${dynamics}" />
     </joint>
-    <xacro:link_with_sc no_prefix="${no_prefix}" name="link7" gazebo="${gazebo}" rpy="0 0 ${pi/4}" with_sc="${with_sc}" with_accelerometers="false">
+    <xacro:link_with_sc no_prefix="${no_prefix}" name="link7" include_self_collision_geometry="${include_self_collision_geometry}" rpy="0 0 ${pi/4}" with_sc="${with_sc}" with_accelerometers="false">
       <self_collision_geometries>
         <xacro:collision_capsule xyz="0 0 0.01" direction="z" radius="${0.04+safety_distance}" length="0.14" />

File: robots/common/franka_robot.xacro (robot description, xacro)
@@ -14,5 +14,5 @@
                       ee_id:=none
                       special_connection:=''
-                      gazebo:='false'
+                      include_self_collision_geometry:='true'
                       with_sc:='false'
                       no_prefix:='false'
@@ -29,5 +29,5 @@
       rpy="${rpy}"
       safety_distance="0.03"
-      gazebo="${gazebo}"
+      include_self_collision_geometry="${include_self_collision_geometry}"
       with_sc="${with_sc}"
       connected_to="${connected_to}"
@@ -56,5 +56,5 @@
         tcp_rpy="${tcp_rpy}"
         safety_distance="${safety_distance}"
-        gazebo="${gazebo}"
+        include_self_collision_geometry="${include_self_collision_geometry}"
         description_pkg="${description_pkg}"
         with_sc="${with_sc}"
@@ -77,68 +77,9 @@
         tcp_rpy="${tcp_rpy}"
         safety_distance="${safety_distance}"
-        gazebo="${gazebo}"
+        include_self_collision_geometry="${include_self_collision_geometry}"
         description_pkg="${description_pkg}"
         with_sc="${with_sc}"
       />
     </xacro:if>
-    <!-- Definition of additional Gazebo tags -->
-    <xacro:if value="${gazebo}">
-      <xacro:gazebo-joint joint="${arm_prefix}${robot_type}_joint1"
-        transmission="hardware_interface/PositionJointInterface"/>
-      <xacro:gazebo-joint joint="${arm_prefix}${robot_type}_joint2"
-        transmission="hardware_interface/PositionJointInterface"/>
-      <xacro:gazebo-joint joint="${arm_prefix}${robot_type}_joint3"
-        transmission="hardware_interface/PositionJointInterface"/>
-      <xacro:gazebo-joint joint="${arm_prefix}${robot_type}_joint4"
-        transmission="hardware_interface/PositionJointInterface"/>
-      <xacro:gazebo-joint joint="${arm_prefix}${robot_type}_joint5"
-        transmission="hardware_interface/PositionJointInterface"/>
-      <xacro:gazebo-joint joint="${arm_prefix}${robot_type}_joint6"
-        transmission="hardware_interface/PositionJointInterface"/>
-      <xacro:gazebo-joint joint="${arm_prefix}${robot_type}_joint7"
-        transmission="hardware_interface/PositionJointInterface"/>
-      <xacro:gazebo-joint joint="${arm_prefix}${robot_type}_joint1"
-        transmission="hardware_interface/VelocityJointInterface"/>
-      <xacro:gazebo-joint joint="${arm_prefix}${robot_type}_joint2"
-        transmission="hardware_interface/VelocityJointInterface"/>
-      <xacro:gazebo-joint joint="${arm_prefix}${robot_type}_joint3"
-        transmission="hardware_interface/VelocityJointInterface"/>
-      <xacro:gazebo-joint joint="${arm_prefix}${robot_type}_joint4"
-        transmission="hardware_interface/VelocityJointInterface"/>
-      <xacro:gazebo-joint joint="${arm_prefix}${robot_type}_joint5"
-        transmission="hardware_interface/VelocityJointInterface"/>
-      <xacro:gazebo-joint joint="${arm_prefix}${robot_type}_joint6"
-        transmission="hardware_interface/VelocityJointInterface"/>
-      <xacro:gazebo-joint joint="${arm_prefix}${robot_type}_joint7"
-        transmission="hardware_interface/VelocityJointInterface"/>
-      <xacro:gazebo-joint joint="${arm_prefix}${robot_type}_joint1"
-        transmission="hardware_interface/EffortJointInterface"/>
-      <xacro:gazebo-joint joint="${arm_prefix}${robot_type}_joint2"
-        transmission="hardware_interface/EffortJointInterface"/>
-      <xacro:gazebo-joint joint="${arm_prefix}${robot_type}_joint3"
-        transmission="hardware_interface/EffortJointInterface"/>
-      <xacro:gazebo-joint joint="${arm_prefix}${robot_type}_joint4"
-        transmission="hardware_interface/EffortJointInterface"/>
-      <xacro:gazebo-joint joint="${arm_prefix}${robot_type}_joint5"
-        transmission="hardware_interface/EffortJointInterface"/>
-      <xacro:gazebo-joint joint="${arm_prefix}${robot_type}_joint6"
-        transmission="hardware_interface/EffortJointInterface"/>
-      <xacro:gazebo-joint joint="${arm_prefix}${robot_type}_joint7"
-        transmission="hardware_interface/EffortJointInterface"/>
-      <xacro:transmission-franka-state robot_type="${robot_type}"/>
-      <xacro:transmission-franka-model robot_type="${robot_type}"
-        root="${arm_prefix}${robot_type}_joint1"
-        tip="${arm_prefix}${robot_type}_joint8"
-      />
-      <xacro:if value="${ee_id == 'franka_hand'}">
-        <xacro:gazebo-joint joint="${arm_prefix}${robot_type}_finger_joint1"
-          transmission="hardware_interface/EffortJointInterface"/>
-        <xacro:gazebo-joint joint="${arm_prefix}${robot_type}_finger_joint2"
-          transmission="hardware_interface/EffortJointInterface"/>
-        <!-- Friction specific material for Rubber/Rubber contact -->
-        <xacro:gazebo-friction link="${arm_prefix}${robot_type}_leftfinger" mu="1.13"/>
-        <xacro:gazebo-friction link="${arm_prefix}${robot_type}_rightfinger" mu="1.13"/>
-      </xacro:if>
-    </xacro:if>
   </xacro:macro>
 </robot>
