Commit message: refactor: Remove gazebo tags/macros/args from franka_description
Make the description package simulator-agnostic. All gazebo SDF and
transmission machinery, the gazebo world anchor, and the gazebo-specific
self-collision suppression are removed; the gazebo:=false argument and the
gazebo_ros export are dropped throughout robots, end_effectors and the URDF
generation workflow.

Self-collision geometry is now gated by the include_self_collision_geometry
capability flag instead of a gazebo toggle. The removed gazebo content is
relocated to franka_gazebo, which owns the simulator-specific blocks.

The removal of the public gazebo xacro argument is recorded in a CHANGELOG
UNRELEASED migration note: consumers that passed gazebo:=true must now use
the franka_gazebo bringup entry points; the old argument is inert.

Behavior-preserving: URDF expansions are byte-identical to before.

File: robots/common/utils.xacro (robot description, xacro)
@@ -26,11 +26,13 @@
   <!--  * detailed meshes for environmental collision checking    -->
   <!--  * and coarse geometry models for self-collision checking  -->
-  <!--    (only if 'gazebo' param is set)                         -->
+  <!--    (only if 'include_self_collision_geometry' is true)     -->
   <!--                                                            -->
   <!-- name:  Name of the robot link (without prefix)             -->
   <!-- rpy:   Rotation of the *_sc link relative to parent [rad]  -->
   <!-- self_collision_geometries:  self <collision> models        -->
+  <!-- include_self_collision_geometry: emit the coarse capsules  -->
+  <!--   inside the *_sc sub-link (true) or leave it empty (false) -->
   <!-- ========================================================== -->
-  <xacro:macro name="link_with_sc" params="name no_prefix:='false' rpy:='0 0 0' **self_collision_geometries gazebo:=false with_sc:=false with_accelerometers:=false">
+  <xacro:macro name="link_with_sc" params="name no_prefix:='false' rpy:='0 0 0' **self_collision_geometries include_self_collision_geometry:=true with_sc:=false with_accelerometers:=false">
     <xacro:property name="prefix" value="${'' if no_prefix else arm_prefix + robot_type + '_'}" />
     <!-- sub-link defining detailed meshes for collision with environment -->
@@ -51,7 +53,7 @@
     <xacro:if value="${with_sc}">
       <link name="${prefix}${name}_sc">
-        <xacro:unless value="${gazebo}">
+        <xacro:if value="${include_self_collision_geometry}">
           <xacro:insert_block name="self_collision_geometries" />
-        </xacro:unless>
+        </xacro:if>
       </link>
       <!-- fixed joint between both sub-links -->
@@ -106,98 +108,4 @@
       </geometry>
     </collision>
-  </xacro:macro>
-  <!-- ========================================================== -->
-  <!-- Adds the required tags to simulate one joint in gazebo     -->
-  <!--                                                            -->
-  <!-- joint - Name of the fer joint to simulate                  -->
-  <!-- transmission - type of the transmission of the joint       -->
-  <!-- ========================================================== -->
-  <xacro:macro name="gazebo-joint" params="joint transmission:=hardware_interface/EffortJointInterface">
-    <gazebo reference="${joint}">
-      <!-- Needed for ODE to output external wrenches on joints -->
-      <provideFeedback>true</provideFeedback>
-    </gazebo>
-    <transmission name="${joint}_transmission">
-      <type>transmission_interface/SimpleTransmission</type>
-      <joint name="${joint}">
-        <hardwareInterface>${transmission}</hardwareInterface>
-      </joint>
-      <actuator name="${joint}_motor">
-        <hardwareInterface>${transmission}</hardwareInterface>
-      </actuator>
-    </transmission>
-  </xacro:macro>
-  <xacro:macro name="gazebo-friction" params="link mu">
-    <gazebo reference="${link}">
-      <collision>
-        <max_contacts>10</max_contacts>
-        <surface>
-          <contact>
-            <ode>
-              <!-- These two parameter need application specific tuning. -->
-              <!-- Usually you want no "snap out" velocity and a generous -->
-              <!-- penetration depth to keep the grasping stable -->
-              <max_vel>0</max_vel>
-              <min_depth>0.001</min_depth>
-            </ode>
-          </contact>
-          <friction>
-            <ode>
-              <mu>${mu}</mu>
-              <mu2>${mu}</mu2>
-            </ode>
-          </friction>
-          <bounce/>
-        </surface>
-      </collision>
-    </gazebo>
-  </xacro:macro>
-  <!-- ========================================================== -->
-  <!-- Adds the required tags to provide a `FrankaStateInterface` -->
-  <!-- when simulating with franka_hw_sim plugin                  -->
-  <!--                                                            -->
-  <!-- robot_type - Arm ID of the fer to simulate (default 'fer')     -->
-  <!-- ========================================================== -->
-  <xacro:macro name="transmission-franka-state" params="robot_type:=fer">
-    <transmission name="${arm_prefix}${robot_type}_franka_state">
-      <type>franka_hw/FrankaStateInterface</type>
-      <joint name="${arm_prefix}${robot_type}_joint1"><hardwareInterface>franka_hw/FrankaStateInterface</hardwareInterface></joint>
-      <joint name="${arm_prefix}${robot_type}_joint2"><hardwareInterface>franka_hw/FrankaStateInterface</hardwareInterface></joint>
-      <joint name="${arm_prefix}${robot_type}_joint3"><hardwareInterface>franka_hw/FrankaStateInterface</hardwareInterface></joint>
-      <joint name="${arm_prefix}${robot_type}_joint4"><hardwareInterface>franka_hw/FrankaStateInterface</hardwareInterface></joint>
-      <joint name="${arm_prefix}${robot_type}_joint5"><hardwareInterface>franka_hw/FrankaStateInterface</hardwareInterface></joint>
-      <joint name="${arm_prefix}${robot_type}_joint6"><hardwareInterface>franka_hw/FrankaStateInterface</hardwareInterface></joint>
-      <joint name="${arm_prefix}${robot_type}_joint7"><hardwareInterface>franka_hw/FrankaStateInterface</hardwareInterface></joint>
-      <actuator name="${arm_prefix}${robot_type}_motor1"><hardwareInterface>franka_hw/FrankaStateInterface</hardwareInterface></actuator>
-      <actuator name="${arm_prefix}${robot_type}_motor2"><hardwareInterface>franka_hw/FrankaStateInterface</hardwareInterface></actuator>
-      <actuator name="${arm_prefix}${robot_type}_motor3"><hardwareInterface>franka_hw/FrankaStateInterface</hardwareInterface></actuator>
-      <actuator name="${arm_prefix}${robot_type}_motor4"><hardwareInterface>franka_hw/FrankaStateInterface</hardwareInterface></actuator>
-      <actuator name="${arm_prefix}${robot_type}_motor5"><hardwareInterface>franka_hw/FrankaStateInterface</hardwareInterface></actuator>
-      <actuator name="${arm_prefix}${robot_type}_motor6"><hardwareInterface>franka_hw/FrankaStateInterface</hardwareInterface></actuator>
-      <actuator name="${arm_prefix}${robot_type}_motor7"><hardwareInterface>franka_hw/FrankaStateInterface</hardwareInterface></actuator>
-    </transmission>
-  </xacro:macro>
-  <!-- ============================================================ -->
-  <!-- Adds the required tags to provide a `FrankaModelInterface`   -->
-  <!-- when simulating with franka_hw_sim plugin                    -->
-  <!--                                                              -->
-  <!-- robot_type - Arm ID of the fer to simulate (default 'fer')       -->
-  <!-- root   - Joint name of the base of the robot                 -->
-  <!-- tip    - Joint name of the tip of the robot (flange or hand) -->
-  <!-- ============================================================ -->
-  <xacro:macro name="transmission-franka-model" params="robot_type:=fer root:=fer_joint1 tip:=fer_joint7">
-    <transmission name="${arm_prefix}${robot_type}_franka_model">
-      <type>franka_hw/FrankaModelInterface</type>
-      <joint name="${root}">
-        <role>root</role>
-        <hardwareInterface>franka_hw/FrankaModelInterface</hardwareInterface>
-      </joint>
-      <joint name="${tip}">
-        <role>tip</role>
-        <hardwareInterface>franka_hw/FrankaModelInterface</hardwareInterface>
-      </joint>
-      <actuator name="${root}_motor_root"><hardwareInterface>franka_hw/FrankaModelInterface</hardwareInterface></actuator>
-      <actuator name="${tip}_motor_tip"  ><hardwareInterface>franka_hw/FrankaModelInterface</hardwareInterface></actuator>
-    </transmission>
   </xacro:macro>
   <xacro:macro name="inertia-cylinder" params="mass radius h">

File: robots/fer/fer.urdf.xacro (robot description, xacro)
@@ -27,6 +27,8 @@
   <!-- Should self-collision be enabled? -->
   <xacro:arg name="with_sc" default="false"/>
-  <!-- Should the robot be spawned in Gazebo?" -->
-  <xacro:arg name="gazebo" default="false"/>
+  <!-- The frame the robot base is rigidly attached to -->
+  <xacro:arg name="connected_to" default="base"/>
+  <!-- Emit the coarse self-collision capsule geometry inside the *_sc sub-links? -->
+  <xacro:arg name="include_self_collision_geometry" default="true"/>
   <!-- Name of the description package -->
   <xacro:arg name="description_pkg" default="franka_description"/>
@@ -40,14 +42,6 @@
   offset with respect to the world-->
   <xacro:arg name="rpy" default="0 0 0"/>
-  <xacro:if value="$(arg gazebo)">
-    <link name="world"/>
-    <joint name="world_joint" type="fixed">
-      <origin xyz="$(arg xyz)" rpy="$(arg rpy)"/>
-      <parent link="world"/>
-      <child link="${modified_prefix}$(arg robot_type)_link0"/>
-    </joint>
-  </xacro:if>
   <xacro:franka_robot robot_type="fer"
-    gazebo="$(arg gazebo)"
+    include_self_collision_geometry="$(arg include_self_collision_geometry)"
     hand="$(arg hand)"
     ee_id="$(arg ee_id)"
@@ -62,5 +56,5 @@
     arm_prefix="${modified_prefix}"
     description_pkg="$(arg description_pkg)"
-    connected_to="base">
+    connected_to="$(arg connected_to)">
   </xacro:franka_robot>
 </robot>

File: robots/fp3/fp3.urdf.xacro (robot description, xacro)
@@ -27,6 +27,8 @@
   <!-- Should self-collision be enabled? -->
   <xacro:arg name="with_sc" default="false"/>
-  <!-- Should the robot be spawned in Gazebo?" -->
-  <xacro:arg name="gazebo" default="false"/>
+  <!-- The frame the robot base is rigidly attached to -->
+  <xacro:arg name="connected_to" default="base"/>
+  <!-- Emit the coarse self-collision capsule geometry inside the *_sc sub-links? -->
+  <xacro:arg name="include_self_collision_geometry" default="true"/>
   <!-- Name of the description package -->
   <xacro:arg name="description_pkg" default="franka_description"/>
@@ -40,14 +42,6 @@
   offset with respect to the world-->
   <xacro:arg name="rpy" default="0 0 0"/>
-  <xacro:if value="$(arg gazebo)">
-    <link name="world"/>
-    <joint name="world_joint" type="fixed">
-      <origin xyz="$(arg xyz)" rpy="$(arg rpy)"/>
-      <parent link="world"/>
-      <child link="${modified_prefix}$(arg robot_type)_link0"/>
-    </joint>
-  </xacro:if>
   <xacro:franka_robot robot_type="fp3"
-    gazebo="$(arg gazebo)"
+    include_self_collision_geometry="$(arg include_self_collision_geometry)"
     hand="$(arg hand)"
     ee_id="$(arg ee_id)"
@@ -62,5 +56,5 @@
     arm_prefix="${modified_prefix}"
     description_pkg="$(arg description_pkg)"
-    connected_to="base">
+    connected_to="$(arg connected_to)">
   </xacro:franka_robot>
 </robot>

File: robots/fr3/fr3.urdf.xacro (robot description, xacro)
@@ -27,6 +27,8 @@
   <!-- Should self-collision be enabled? -->
   <xacro:arg name="with_sc" default="false"/>
-  <!-- Should the robot be spawned in Gazebo?" -->
-  <xacro:arg name="gazebo" default="false"/>
+  <!-- The frame the robot base is rigidly attached to -->
+  <xacro:arg name="connected_to" default="base"/>
+  <!-- Emit the coarse self-collision capsule geometry inside the *_sc sub-links? -->
+  <xacro:arg name="include_self_collision_geometry" default="true"/>
   <!-- Name of the description package -->
   <xacro:arg name="description_pkg" default="franka_description"/>
@@ -40,14 +42,6 @@
   offset with respect to the world-->
   <xacro:arg name="rpy" default="0 0 0"/>
-  <xacro:if value="$(arg gazebo)">
-    <link name="world"/>
-    <joint name="world_joint" type="fixed">
-      <origin xyz="$(arg xyz)" rpy="$(arg rpy)"/>
-      <parent link="world"/>
-      <child link="${modified_prefix}$(arg robot_type)_link0"/>
-    </joint>
-  </xacro:if>
   <xacro:franka_robot robot_type="fr3"
-    gazebo="$(arg gazebo)"
+    include_self_collision_geometry="$(arg include_self_collision_geometry)"
     hand="$(arg hand)"
     ee_id="$(arg ee_id)"
@@ -62,5 +56,5 @@
     arm_prefix="${modified_prefix}"
     description_pkg="$(arg description_pkg)"
-    connected_to="base">
+    connected_to="$(arg connected_to)">
   </xacro:franka_robot>
 </robot>

File: robots/fr3_duo/fr3_duo.urdf.xacro (robot description, xacro)
@@ -26,6 +26,6 @@
   <!-- Should self-collision be enabled? -->
   <xacro:arg name="with_sc" default="false"/>
-  <!-- Should the robot be spawned in Gazebo?" -->
-  <xacro:arg name="gazebo" default="false"/>
+  <!-- Emit the coarse self-collision capsule geometry inside the *_sc sub-links? -->
+  <xacro:arg name="include_self_collision_geometry" default="true"/>
   <!-- Name of the description package -->
   <xacro:arg name="description_pkg" default="franka_description"/>
@@ -40,12 +40,4 @@
   <xacro:arg name="base_mount" default="base"/>
   <xacro:property name="base_mount_str" value="$(arg base_mount)"/>
-  <xacro:if value="$(arg gazebo)">
-    <link name="world"/>
-    <joint name="world_joint" type="fixed">
-      <origin xyz="$(arg xyz)" rpy="$(arg rpy)"/>
-      <parent link="world"/>
-      <child link="${base_mount_str}"/>
-    </joint>
-  </xacro:if>
   <xacro:if value="${base_mount_str == 'base'}">
     <link name="${base_mount_str}"/>
@@ -62,9 +54,12 @@
     safety_distance="$(arg safety_distance)"
     with_sc="$(arg with_sc)"
-    gazebo="$(arg gazebo)"
+    include_self_collision_geometry="$(arg include_self_collision_geometry)"
     description_pkg="$(arg description_pkg)"
     base_mount="${base_mount_str}"
     connected_to="${base_mount_str}"
     arm_prefixes="${arm_prefixes_list}"
-    no_prefix="$(arg no_prefix)"/>
+    no_prefix="$(arg no_prefix)">
+    <arm0_extras/>
+    <arm1_extras/>
+  </xacro:fr3_duo>
 </robot>

File: robots/fr3_duo/fr3_duo.xacro (robot description, xacro)
@@ -17,5 +17,5 @@
             safety_distance
             with_sc
-            gazebo
+            include_self_collision_geometry
             description_pkg
             base_mount
@@ -23,5 +23,7 @@
             arm_prefixes
             no_prefix:=false
-            is_mobile_fr3_duo:=false">
+            is_mobile_fr3_duo:=false
+            **arm0_extras
+            **arm1_extras">
     <xacro:property name="robot_types_list" value="${robot_types}"/>
     <xacro:property name="arm_prefixes_list" value="${arm_prefixes}"/>
@@ -47,5 +49,5 @@
         <xacro:franka_robot
           robot_type="${robot_type_i}"
-          gazebo="${gazebo}"
+          include_self_collision_geometry="${include_self_collision_geometry}"
           hand="${hand}"
           ee_id="${ee_id}"
@@ -62,4 +64,13 @@
           connected_to="${arm_prefixes_list[i]}_base">
         </xacro:franka_robot>
+        <!-- Per-arm extension point (e.g. simulation transmissions injected by
+             the simulation bringup). Each block is evaluated in the caller's
+             scope, so the caller supplies the concrete arm prefix / robot type. -->
+        <xacro:if value="${i == 0}">
+          <xacro:insert_block name="arm0_extras"/>
+        </xacro:if>
+        <xacro:if value="${i == 1}">
+          <xacro:insert_block name="arm1_extras"/>
+        </xacro:if>
         <xacro:fr3_duo_loop i="${i+1}"/>
       </xacro:unless>

File: robots/fr3v2/fr3v2.urdf.xacro (robot description, xacro)
@@ -27,6 +27,8 @@
   <!-- Should self-collision be enabled? -->
   <xacro:arg name="with_sc" default="false"/>
-  <!-- Should the robot be spawned in Gazebo?" -->
-  <xacro:arg name="gazebo" default="false"/>
+  <!-- The frame the robot base is rigidly attached to -->
+  <xacro:arg name="connected_to" default="base"/>
+  <!-- Emit the coarse self-collision capsule geometry inside the *_sc sub-links? -->
+  <xacro:arg name="include_self_collision_geometry" default="true"/>
   <!-- Name of the description package -->
   <xacro:arg name="description_pkg" default="franka_description"/>
@@ -40,14 +42,6 @@
   offset with respect to the world-->
   <xacro:arg name="rpy" default="0 0 0"/>
-  <xacro:if value="$(arg gazebo)">
-    <link name="world"/>
-    <joint name="world_joint" type="fixed">
-      <origin xyz="$(arg xyz)" rpy="$(arg rpy)"/>
-      <parent link="world"/>
-      <child link="${modified_prefix}$(arg robot_type)_link0"/>
-    </joint>
-  </xacro:if>
   <xacro:franka_robot robot_type="fr3v2"
-    gazebo="$(arg gazebo)"
+    include_self_collision_geometry="$(arg include_self_collision_geometry)"
     hand="$(arg hand)"
     ee_id="$(arg ee_id)"
@@ -62,5 +56,5 @@
     arm_prefix="${modified_prefix}"
     description_pkg="$(arg description_pkg)"
-    connected_to="base">
+    connected_to="$(arg connected_to)">
   </xacro:franka_robot>
 </robot>

File: robots/fr3v2_1/fr3v2_1.urdf.xacro (robot description, xacro)
@@ -27,6 +27,8 @@
   <!-- Should self-collision be enabled? -->
   <xacro:arg name="with_sc" default="false"/>
-  <!-- Should the robot be spawned in Gazebo?" -->
-  <xacro:arg name="gazebo" default="false"/>
+  <!-- The frame the robot base is rigidly attached to -->
+  <xacro:arg name="connected_to" default="base"/>
+  <!-- Emit the coarse self-collision capsule geometry inside the *_sc sub-links? -->
+  <xacro:arg name="include_self_collision_geometry" default="true"/>
   <!-- Name of the description package -->
   <xacro:arg name="description_pkg" default="franka_description"/>
@@ -40,14 +42,6 @@
   offset with respect to the world-->
   <xacro:arg name="rpy" default="0 0 0"/>
-  <xacro:if value="$(arg gazebo)">
-    <link name="world"/>
-    <joint name="world_joint" type="fixed">
-      <origin xyz="$(arg xyz)" rpy="$(arg rpy)"/>
-      <parent link="world"/>
-      <child link="${modified_prefix}$(arg robot_type)_link0"/>
-    </joint>
-  </xacro:if>
   <xacro:franka_robot robot_type="fr3v2_1"
-    gazebo="$(arg gazebo)"
+    include_self_collision_geometry="$(arg include_self_collision_geometry)"
     hand="$(arg hand)"
     ee_id="$(arg ee_id)"
@@ -62,5 +56,5 @@
     arm_prefix="${modified_prefix}"
     description_pkg="$(arg description_pkg)"
-    connected_to="base">
+    connected_to="$(arg connected_to)">
   </xacro:franka_robot>
 </robot>

File: robots/mobile_fr3_duo_v0_2/mobile_fr3_duo_v0_2.urdf.xacro (robot description, xacro)
@@ -26,6 +26,6 @@
   <!-- Should self-collision be enabled? -->
   <xacro:arg name="with_sc" default="false"/>
-  <!-- Should the robot be spawned in Gazebo?" -->
-  <xacro:arg name="gazebo" default="false"/>
+  <!-- Emit the coarse self-collision capsule geometry inside the *_sc sub-links? -->
+  <xacro:arg name="include_self_collision_geometry" default="true"/>
   <!-- Name of the description package -->
   <xacro:arg name="description_pkg" default="franka_description"/>
@@ -39,5 +39,4 @@
     robot_types="$(arg robot_types)"
     hand="$(arg hand)"
-    gazebo="$(arg gazebo)"
     reduced_version="$(arg reduced_version)"
     description_pkg="$(arg description_pkg)"
@@ -52,4 +51,8 @@
     tcp_rpy="$(arg tcp_rpy)"
     safety_distance="$(arg safety_distance)"
-    with_sc="$(arg with_sc)"/>
+    with_sc="$(arg with_sc)"
+    include_self_collision_geometry="$(arg include_self_collision_geometry)">
+    <arm0_extras/>
+    <arm1_extras/>
+  </xacro:mobile_fr3_duo_v0_2>
 </robot>

File: robots/mobile_fr3_duo_v0_2/mobile_fr3_duo_v0_2.xacro (robot description, xacro)
@@ -5,5 +5,5 @@
     params="robot_types
             hand
-            gazebo
+            include_self_collision_geometry
             reduced_version
             description_pkg
@@ -18,5 +18,7 @@
             tcp_rpy
             safety_distance
-            with_sc">
+            with_sc
+            **arm0_extras
+            **arm1_extras">
     <xacro:include filename="$(find franka_description)/accessories/franka_spine_v0_1/franka_spine.xacro"/>
     <xacro:include filename="$(find franka_description)/robots/common/franka_robot.xacro"/>
@@ -40,6 +42,5 @@
     <xacro:tmrv0_2
       mobile_robot_type="${robot_types_list[0]}"
-      reduced_version="${reduced_version}"
-      gazebo="${gazebo}"/>
+      reduced_version="${reduced_version}"/>
     <!-- Spine -->
     <xacro:franka_spine parent="base_link"/>
@@ -58,10 +59,13 @@
       safety_distance="${safety_distance}"
       with_sc="${with_sc}"
-      gazebo="${gazebo}"
+      include_self_collision_geometry="${include_self_collision_geometry}"
       description_pkg="${description_pkg}"
       base_mount="franka_spine_mounting_point"
       connected_to="${connected_to}"
       arm_prefixes="${arm_prefixes_list}"
-      is_mobile_fr3_duo="true"/>
+      is_mobile_fr3_duo="true">
+      <arm0_extras><xacro:insert_block name="arm0_extras"/></arm0_extras>
+      <arm1_extras><xacro:insert_block name="arm1_extras"/></arm1_extras>
+    </xacro:fr3_duo>
   </xacro:macro>
 </robot>

File: robots/tmrv0_2/tmrv0_2.urdf.xacro (robot description, xacro)
@@ -11,6 +11,4 @@
   <!-- Should the reduced kinematic version (without caster wheels) be used? -->
   <xacro:arg name="reduced_version" default="false"/>
-  <!-- Should the robot be spawned in Gazebo?" -->
-  <xacro:arg name="gazebo" default="false"/>
   <!-- The namespace of the robot -->
   <xacro:arg name="robot_namespace" default=""/>
@@ -20,5 +18,4 @@
   <xacro:tmrv0_2 mobile_robot_type="$(arg robot_type)"
     reduced_version="$(arg reduced_version)"
-    robot_namespace="$(arg robot_namespace)"
-    gazebo="$(arg gazebo)"/>
+    robot_namespace="$(arg robot_namespace)"/>
 </robot>

File: robots/tmrv0_2/tmrv0_2.xacro (robot description, xacro)
@@ -4,6 +4,5 @@
     params="mobile_robot_type
                   reduced_version:=false
-                  robot_namespace:=''
-                  gazebo:=false">
+                  robot_namespace:=''">
     <xacro:include filename="$(find franka_description)/robots/tmrv0_2/argo_drive.xacro"/>
     <xacro:include filename="$(find franka_description)/robots/tmrv0_2/caster_wheel.xacro"/>
