Commit message: fix: define modified_prefix in tmrv0_2 description for mobile_teleop
The shared bringup franka_arm.urdf.xacro passes arm_prefix="${modified_prefix}"
to the franka_arm_ros2_control macro, but tmrv0_2.urdf.xacro was the only
robot description not defining the file-scope modified_prefix property. As a
result mobile_teleop.launch.py (robot_type: tmrv0_2) failed with
'name 'modified_prefix' is not defined'.

Add the arm_prefix arg plus prefix/modified_prefix properties to match the
established arm-description pattern; the mobile base links are intentionally
left unprefixed.

File: robots/tmrv0_2/tmrv0_2.urdf.xacro (robot description, xacro)
@@ -5,4 +5,8 @@
   <!-- The ID of the robot model to be used -->
   <xacro:arg name="robot_type" default="tmrv0_2"/>
+  <!-- The prefix of the robot. arm_prefix exists only to satisfy the shared
+       franka_arm bringup macro (modified_prefix); the mobile base links are
+       intentionally left unprefixed. -->
+  <xacro:arg name="arm_prefix" default=""/>
   <!-- Should the reduced kinematic version (without caster wheels) be used? -->
   <xacro:arg name="reduced_version" default="false"/>
@@ -11,4 +15,7 @@
   <!-- The namespace of the robot -->
   <xacro:arg name="robot_namespace" default=""/>
+  <!-- Append an underscore to the user-provided prefix, if non-empty. -->
+  <xacro:property name="prefix" value="$(arg arm_prefix)"/>
+  <xacro:property name="modified_prefix" value="${prefix + '_' if prefix else ''}"/>
   <xacro:tmrv0_2 mobile_robot_type="$(arg robot_type)"
     reduced_version="$(arg reduced_version)"
