Commit message: fix: apply no_prefix to the end effector as well as the arm
franka_arm dropped the prefix from its link names under no_prefix but
franka_robot still attached the end effector to <robot_type>_link8 and let
the end effector prefix itself, so the two halves of the robot stopped
referring to each other: every no_prefix description carrying an end
effector named a parent link the urdf did not define and was rejected by
the urdf parser, while the srdf, which does honour no_prefix, named end
effector links the urdf did not have.

franka_hand already declared a no_prefix parameter it never read, so this
wires up what was intended rather than introducing a new concept.

The macro's own default was the quoted string 'false', which is truthy in
python; it has to be a real boolean now that it decides the link prefix,
otherwise direct callers of the macro would silently lose it.

On main 20 of the 116 generated urdf variants fail check_urdf, all of them
no_prefix combined with an end effector. All 116 pass here, and the only
generated output that changes is those 20 previously unloadable ones.

Signed-off-by: Kamal Mohy El Dine <kamal.mohy@franka.de>

File: end_effectors/common/ee_with_one_link.xacro (robot description, xacro)
@@ -2,8 +2,8 @@
 <robot xmlns:xacro="http://www.ros.org/wiki/xacro" name="ee_with_one_link">
   <!-- safety_distance: Minimum safety distance in [m] by which the collision volumes are expanded and which is enforced during robot motions -->
-  <xacro:macro name="ee_with_one_link" params="connected_to:='' robot_type arm_prefix:='' ee_id ee_inertials rpy_ee:='0 0 0' xyz_ee:='0 0 0' tcp_xyz:='0 0 0' tcp_rpy:='0 0 0' safety_distance:=0 include_self_collision_geometry:=true description_pkg:=franka_description with_sc:=false">
+  <xacro:macro name="ee_with_one_link" params="connected_to:='' robot_type arm_prefix:='' ee_id ee_inertials rpy_ee:='0 0 0' xyz_ee:='0 0 0' tcp_xyz:='0 0 0' tcp_rpy:='0 0 0' safety_distance:=0 include_self_collision_geometry:=true description_pkg:=franka_description with_sc:=false no_prefix:=false">
     <xacro:property name="ee_prefix" default="robot_"/>
     <xacro:unless value="${robot_type == ''}">
-      <xacro:property name="ee_prefix" value="${arm_prefix}${robot_type}_" />
+      <xacro:property name="ee_prefix" value="${'' if no_prefix else arm_prefix + robot_type + '_'}" />
     </xacro:unless>
     <xacro:unless value="${connected_to == ''}">

File: end_effectors/common/franka_hand.xacro (robot description, xacro)
@@ -17,5 +17,5 @@
     <xacro:property name="ee_prefix" default="robot_"/>
     <xacro:unless value="${robot_type == ''}">
-      <xacro:property name="ee_prefix" value="${arm_prefix}${robot_type}_" />
+      <xacro:property name="ee_prefix" value="${'' if no_prefix else arm_prefix + robot_type + '_'}" />
     </xacro:unless>
     <xacro:unless value="${connected_to == ''}">

File: robots/common/franka_robot.xacro (robot description, xacro)
@@ -16,5 +16,5 @@
                       include_self_collision_geometry:='true'
                       with_sc:='false'
-                      no_prefix:='false'
+                      no_prefix:=false
                       arm_prefix:=''
                       description_pkg:='franka_description'
@@ -29,4 +29,8 @@
       value="${'0 0 0.1034' if ee_id == 'franka_hand' else '0 0 0.105' if ee_id == 'cobot_pump' else '0 0 0'}"/>
     <xacro:property name="tcp_xyz_resolved" value="${ee_tcp_xyz if tcp_xyz == '' else tcp_xyz}"/>
+    <!-- franka_arm derives its link names this way, so the end effector has to attach to
+         the same names and prefix itself the same way, or the two halves of the robot do
+         not reference each other. -->
+    <xacro:property name="link_prefix" value="${'' if no_prefix else arm_prefix + robot_type + '_'}"/>
     <xacro:franka_arm
       robot_type="${robot_type}"
@@ -51,9 +55,10 @@
       </xacro:if>
       <xacro:property name="connection"
-        value="${special_connection if special_connection != '' else robot_type + '_link8'}"/>
+        value="${arm_prefix + special_connection if special_connection != '' else link_prefix + 'link8'}"/>
       <xacro:franka_hand
-        connected_to="${arm_prefix}${connection}"
+        connected_to="${connection}"
         robot_type="${robot_type}"
         arm_prefix="${arm_prefix}"
+        no_prefix="${no_prefix}"
         ee_id="${ee_id}_${ee_color}"
         ee_inertials="${xacro.load_yaml('$(find franka_description)/end_effectors/' + ee_id + '/inertials.yaml')}"
@@ -72,9 +77,10 @@
       <xacro:include filename="$(find franka_description)/end_effectors/common/utils.xacro"/>
       <xacro:property name="connection"
-        value="${special_connection if special_connection != '' else robot_type + '_link8'}"/>
+        value="${arm_prefix + special_connection if special_connection != '' else link_prefix + 'link8'}"/>
       <xacro:ee_with_one_link
-        connected_to="${arm_prefix}${connection}"
+        connected_to="${connection}"
         robot_type="${robot_type}"
         arm_prefix="${arm_prefix}"
+        no_prefix="${no_prefix}"
         ee_id="${ee_id}"
         ee_inertials="${xacro.load_yaml('$(find franka_description)/end_effectors/' + ee_id + '/inertials.yaml')}"
